File: boards/encoder/encoder.kicad_sch (KiCad schematic)
At the start: 0 parts

Commit message: v0.1
Parts:
- added C1, C2, C3, C4: C, symbol Device:C
- added L1: L, symbol Device:L
- added R1, R2, R3: R, symbol Device:R
- added SW1: SW_Push, Button_Switch_SMD:SW_MEC_5GSH9, symbol Switch:SW_Push
- added U1: MSPM0G310x, RHB0032D-IPC_A, symbol MCU_Texas_MSP430:MSPM0G310x
- added U2: TPS62A02A, SOT6_DRL_TEX, symbol Regulator_Switching:TPS62A02A
Connections:
- new net: C1.2, R1.2, R2.1, U2.5 (FB)
- new net: L1.1, U2.2 (SW)
- new net +3.3V: C1.1, C2.1, L1.2, R1.1, R3.1, U1.4 (VDD)
- new net BOOT: U1.22 (PA18_A1_3)
- new net GND: C2.2, C3.2, C4.1, R2.2, SW1.2, U1.33 (Thermal_pad), U1.5 (VSS), U2.1 (GND)
- new net PEN: U2.4 (EN)
- new net RESET: C3.1, R3.2, SW1.1, U1.3 (RST_N), U2.6 (PG)
- new net ROSC: U1.6 (PA2_ROSC)
- new net SWCLK: U1.24 (PA20_SWCLK)
- new net SWDIO: U1.23 (PA19_SWDIO)
- new net VCC: C4.2, U2.3 (VIN)
- new net VCORE: U1.32 (VCORE)
- new net VREF+: U1.27 (PA23_VREF+)
- new net VREF-: U1.25 (PA21_A1_7_VREF-)

Commit message: v0.1.1
Parts:
- added C5, C6: C, symbol Device:C
- added R4, R5, R6: R, symbol Device:R
- added SW2, SW3: SW_SPST, symbol Switch:SW_SPST
- added U3: TCAN1044V, SOT-23-THIN-8_DDF_TEX, symbol Interface_CAN_LIN:TCAN1044V
Connections:
- net +3.3V: now also C4.1, R6.2, U3.5 (VIO)
- net BOOT: now also R6.1, SW2.1 (A)
- net GND: now also C4.2, C5.2, C6.2, R4.1, SW2.2 (B), SW3.2 (B), U3.2 (GND); no longer C4.1
- net PEN: now also R5.1, SW3.1 (A)
- net ROSC: now also R4.2
- net VCC: now also C5.1, R5.2, U3.3 (VCC); no longer C4.2
- net VCORE: now also C6.1
- net CAN_TX: now reaches U1.16 (PA12_FCC_IN)
- net CAN_TX: now also U3.1 (TXD)
- net CAN_RX: now reaches U1.17 (PA13)
- net CAN_RX: now also U3.4 (RXD)
- new net CANH: U3.7 (CANH)
- new net CANL: U3.6 (CANL)
- new net STB: U3.8 (STB)
Other:
- moved on the sheet: C3, R3, SW1

Commit message: v0.1.2
Parts:
- added C7: C, symbol Device:C
- added U4: ~, symbol Sensor_Magnetic:CT310
Connections:
- net VREF+: now also C7.1
- net VREF-: now also C7.2
- new net COS+: U4.5 (COS+)
- new net COS-: U4.7 (COS-)
- new net GNDA: U4.4 (GSIN), U4.8 (GCOS)
- new net SIN+: U4.3 (SIN+)
- new net SIN-: U4.1 (SIN-)
- new net VDDA: U4.2 (VSIN), U4.6 (VCOS)
Other:
- moved on the sheet: C1, C2, C3, C4, C5, C6, L1, R1, R2, R3, R4, R5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

Commit message: v0.1.3
Parts:
- added C5: C, symbol Device:C
- renumbered C5 to C2, C2 to C3
Connections:
- net +3.3V: now also C5.1
- net GND: now also C5.2
- net BSL_UART_TX: now reaches U1.14 (PA10_CLK_OUT)
- net BSL_UART_RX: now reaches U1.15 (PA11)
Other:
- moved on the sheet: C2, C3, C4, C6, C7, R3, R5, R6, SW1, SW2, SW3

Commit message: v0.1.4
Parts:
- added U5, U6: INA826, INA826AIDRGR:SON50P300X300X80-9N200X120, symbol Amplifier_Instrumentation:INA826
- U4: value ~ -> CT310
Other:
- moved on the sheet: U4

Commit message: v0.1.5
Connections:
- net SIN+: now also U5.4 (+IN)
- net SIN-: now also U5.1 (-IN)
Changed lines of the file:
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@@
+	(wire
+		(pts
+			(xy 80.01 76.2) (xy 76.2 76.2)
+		)
+		(stroke
+			(width 0)
+			(type default)
+		)
+	)
 	(wire
 		(pts
@@
 		(pts
 			(xy 264.16 115.57) (xy 266.7 115.57)
+		)
+		(stroke
+			(width 0)
+			(type default)
+		)
+	)
+	(wire
+		(pts
+			(xy 76.2 78.74) (xy 80.01 78.74)
 		)
 		(stroke
@@
 	)
 	(label "SIN+"
+		(at 76.2 76.2 180)
+		(effects
+			(font
+				(size 1.27 1.27)
+			)
+			(justify right bottom)
+		)
+	)
+	(label "SIN+"
 		(at 60.96 80.01 0)
 		(effects
@@
 			)
 			(justify left bottom)
+		)
+	)
+	(label "SIN-"
+		(at 76.2 78.74 180)
+		(effects
+			(font
+				(size 1.27 1.27)
+			)
+			(justify right bottom)
 		)
 	)
@@
 		(on_board yes)
 		(dnp no)
-		(fields_autoplaced yes)
 		(property "Reference" "U5"
 			(at 95.25 68.58 0)

Commit message: v0.1.6
Parts:
- added R7, R8: R, symbol Device:R
Connections:
- net COS+: now also U6.4 (+IN)
- net COS-: now also U6.1 (-IN)
- net GNDA: now also U5.5 (GND), U5.9 (EP), U6.5 (GND), U6.9 (EP)
- net VDDA: now also U5.8 (VCC), U6.8 (VCC)
- net at U5.2 (RGA): now also R7.1
- net at U5.3 (RGB): now also R7.2
- net VBIAS: now reaches U5.6 (REF)
- net VBIAS: now also U6.6 (REF)
- net SIND: now reaches U5.7 (VOUT)
- net at U6.2 (RGA): now also R8.1
- net at U6.3 (RGB): now also R8.2
- net COSD: now reaches U6.7 (VOUT)

Commit message: v0.1.7
Parts:
- removed C3: C, symbol Device:C
- removed U3: TCAN1044V, SOT-23-THIN-8_DDF_TEX, symbol Interface_CAN_LIN:TCAN1044V
- added C10, C11, C8: C, symbol Device:C
- added D1, D2, D3: LED, symbol Device:LED
- added J1: US Sensor, symbol Connector_Generic:Conn_01x04
- added J2: SWD, symbol Connector_Generic:Conn_01x04
- added J3: BLS, symbol Connector_Generic:Conn_01x04
- added R10, R11, R12, R13, R14, R15, R9: R, symbol Device:R
Connections:
- net VREF+ is gone; now on net VDDA: C7.1, U1.27 (PA23_VREF+)
- net VREF- is gone; now on net GNDA: C7.2, U1.25 (PA21_A1_7_VREF-)
- net +3.3V: now also D2.2 (A), D3.2 (A), J1.1 (Pin_1)
- net BSL_UART_RX: now also J3.3 (Pin_3)
- net BSL_UART_TX: now also J3.2 (Pin_2)
- net COSD: now also R13.1
- net GND: now also C8.2, J1.2 (Pin_2), J2.4 (Pin_4), J3.4 (Pin_4), R11.2, R14.2
- net GNDA: now also C10.2, C11.2, R10.1
- net RESET: now also C8.1
- net SIND: now also R12.1
- net SWCLK: now also J2.3 (Pin_3)
- net SWDIO: now also J2.2 (Pin_2)
- net VBIAS: now also U1.30 (PA26_A0_1), R10.2, R9.1
- net VDDA: now also R9.2; no longer U5.8 (VCC), U6.8 (VCC)
- net LED_OUT: now reaches U1.1 (PA0_FCC_IN)
- net LED_OUT: now also R15.2
- net SIN_IN: now reaches U1.19 (PA15_A1_0)
- net SIN_IN: now also C10.1, R12.2
- net COS_IN: now reaches U1.31 (PA27_RTC_OUT_A0_0)
- net COS_IN: now also C11.1, R13.2
- net CAN_RX: no longer names the net of U1.17 (PA13)
- net CAN_TX: no longer names the net of U1.16 (PA12_FCC_IN)
- net VCC renamed VDD
- net VDD: now also U5.8 (VCC), U6.8 (VCC), D1.2 (A), J2.1 (Pin_1), J3.1 (Pin_1)
- new net: D3.1 (K), R15.1
- new net: D1.1 (K), R11.1
- new net: D2.1 (K), R14.1
- new net AY_RX: J1.3 (Pin_3)
- new net AY_TX: J1.4 (Pin_4)
Other:
- moved on the sheet: C2, C3, C4, C5, C6, C7, R3, R4, R5, R6, R7, R8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
