File: boards/encoder/encoder.kicad_sch (KiCad schematic)
At the start: 26 parts, among them J1 SWD, J2 Sensore, J3 Sensore, SW1 SW_SPST, SW2 SW_SPST, SW3 SW_Push, U1 MSPM0G310x, U2 M24C08

Commit message: v0.2.3
Parts:
- D3: footprint (none) -> metis-vela:LED_0606_1615Metric
- J1, J2, J3: footprint (none) -> Connector_JST:JST_XH_B4B-XH-A_1x04_P2.50mm_Vertical
- SW1, SW2: footprint (none) -> metis-vela:SW_DS04-254-1-01BK-SMT
- SW3: footprint (none) -> metis-vela:SW_TS04-66-65-BK-260-SMT
Changed lines of the file:
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@@
 			)
 		)
-		(property "Footprint" ""
+		(property "Footprint" "Connector_JST:JST_XH_B4B-XH-A_1x04_P2.50mm_Vertical"
 			(at 102.87 35.56 0)
 			(effects
@@
 			)
 		)
-		(property "Footprint" ""
+		(property "Footprint" "metis-vela:SW_DS04-254-1-01BK-SMT"
 			(at 43.18 130.81 0)
 			(effects
@@
 			)
 		)
-		(property "Footprint" ""
+		(property "Footprint" "metis-vela:LED_0606_1615Metric"
 			(at 87.63 131.572 0)
 			(effects
@@
 			)
 		)
-		(property "Footprint" ""
+		(property "Footprint" "metis-vela:SW_TS04-66-65-BK-260-SMT"
 			(at 71.12 130.81 0)
 			(effects
@@
 			)
 		)
-		(property "Footprint" ""
+		(property "Footprint" "Connector_JST:JST_XH_B4B-XH-A_1x04_P2.50mm_Vertical"
 			(at 161.29 35.56 0)
 			(effects
@@
 			)
 		)
-		(property "Footprint" ""
+		(property "Footprint" "metis-vela:SW_DS04-254-1-01BK-SMT"
 			(at 26.67 130.81 0)
 			(effects
@@
 			)
 		)
-		(property "Footprint" ""
+		(property "Footprint" "Connector_JST:JST_XH_B4B-XH-A_1x04_P2.50mm_Vertical"
 			(at 132.08 35.56 0)
 			(effects

Commit message: v0.2.6
Parts:
- added H1, H2, H3, H4: MountingHole, MountingHole:MountingHole_3.2mm_M3_DIN965_Pad, symbol Mechanical:MountingHole
Connections:
- net COS_IN: now also U1.26 (PA22_A0_7); no longer U1.28 (PA24_A0_3)
- net VDDA_EN: now also U1.28 (PA24_A0_3); no longer U1.9 (PA5_HFXIN_FCC_IN)

Commit message: v0.2.7
Connections:
- net CAN_STB: now also U1.29 (PA25_A0_2); no longer U1.10 (PA6_HFCLK_IN_HFXOUT)
- net ROM_WC: now also U1.9 (PA5_HFXIN_FCC_IN)
- net SIN_IN: now also U1.20 (PA16_A1_1_FCC_IN); no longer U1.19 (PA15_A1_0)
- net VBIAS: now also U1.21 (PA17_A1_2); no longer U1.20 (PA16_A1_1_FCC_IN)
- net VDDA_EN: now also U1.19 (PA15_A1_0); no longer U1.28 (PA24_A0_3)
- no-connect marks 5 -> 4
Changed lines of the file:
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@@
 	)
 	(no_connect
-		(at 207.01 91.44)
+		(at 207.01 63.5)
+	)
+	(no_connect
+		(at 207.01 109.22)
 	)
 	(no_connect
@@
 	)
 	(no_connect
-		(at 207.01 60.96)
-	)
-	(no_connect
 		(at 207.01 78.74)
 	)
-	(no_connect
-		(at 207.01 111.76)
-	)
 	(wire
 		(pts
@@
 	(wire
 		(pts
+			(xy 201.93 88.9) (xy 207.01 88.9)
+		)
+		(stroke
+			(width 0)
+			(type default)
+		)
+	)
+	(wire
+		(pts
 			(xy 201.93 101.6) (xy 207.01 101.6)
 		)
@@
 	(wire
 		(pts
+			(xy 201.93 91.44) (xy 207.01 91.44)
+		)
+		(stroke
+			(width 0)
+			(type default)
+		)
+	)
+	(wire
+		(pts
 			(xy 201.93 93.98) (xy 207.01 93.98)
 		)
@@
 	(wire
 		(pts
+			(xy 201.93 86.36) (xy 207.01 86.36)
+		)
+		(stroke
+			(width 0)
+			(type default)
+		)
+	)
+	(wire
+		(pts
 			(xy 97.79 33.02) (xy 95.25 33.02)
 		)
@@
 	(wire
 		(pts
-			(xy 201.93 63.5) (xy 207.01 63.5)
-		)
-		(stroke
-			(width 0)
-			(type default)
-		)
-	)
-	(wire
-		(pts
 			(xy 57.15 124.46) (xy 57.15 127)
 		)
@@
 	(wire
 		(pts
-			(xy 201.93 109.22) (xy 207.01 109.22)
-		)
-		(stroke
-			(width 0)
-			(type default)
-		)
-	)
-	(wire
-		(pts
 			(xy 86.36 72.39) (xy 91.44 72.39)
 		)
@@
 	(wire
 		(pts
-			(xy 201.93 88.9) (xy 207.01 88.9)
-		)
-		(stroke
-			(width 0)
-			(type default)
-		)
-	)
-	(wire
-		(pts
 			(xy 124.46 40.64) (xy 124.46 43.18)
 		)
@@
 	(wire
 		(pts
+			(xy 201.93 60.96) (xy 207.01 60.96)
+		)
+		(stroke
+			(width 0)
+			(type default)
+		)
+	)
+	(wire
+		(pts
 			(xy 116.84 72.39) (xy 121.92 72.39)
 		)
@@
 	(wire
 		(pts
+			(xy 201.93 111.76) (xy 207.01 111.76)
+		)
+		(stroke
+			(width 0)
+			(type default)
+		)
+	)
+	(wire
+		(pts
 			(xy 133.35 134.62) (xy 133.35 137.16)
 		)
@@
 		(pts
 			(xy 66.04 124.46) (xy 66.04 125.73)
-		)
-		(stroke
-			(width 0)
-			(type default)
-		)
-	)
-	(wire
-		(pts
-			(xy 201.93 86.36) (xy 207.01 86.36)
 		)
 		(stroke
@@
 		)
 	)
-	(label "VBIAS"
-		(at 201.93 88.9 180)
-		(effects
-			(font
-				(size 1.27 1.27)
-			)
-			(justify right bottom)
-		)
-	)
 	(label "LED1_OUT"
 		(at 82.55 140.97 180)
@@
 		)
 	)
+	(label "CAN_STB"
+		(at 201.93 111.76 180)
+		(effects
+			(font
+				(size 1.27 1.27)
+			)
+			(justify right bottom)
+		)
+	)
 	(label "I2C_SCL"
 		(at 201.93 58.42 180)
@@
 		)
 	)
+	(label "VDDA_EN"
+		(at 201.93 86.36 180)
+		(effects
+			(font
+				(size 1.27 1.27)
+			)
+			(justify right bottom)
+		)
+	)
 	(label "VREF+"
 		(at 201.93 106.68 180)
@@
 		)
 	)
+	(label "VBIAS"
+		(at 201.93 91.44 180)
+		(effects
+			(font
+				(size 1.27 1.27)
+			)
+			(justify right bottom)
+		)
+	)
 	(label "RS485_RX"
 		(at 121.92 80.01 0)
@@
 		)
 	)
+	(label "SIN_IN"
+		(at 201.93 88.9 180)
+		(effects
+			(font
+				(size 1.27 1.27)
+			)
+			(justify right bottom)
+		)
+	)
 	(label "VDDA_EN"
 		(at 33.02 69.85 180)
@@
 		)
 	)
-	(label "SIN_IN"
-		(at 201.93 86.36 180)
-		(effects
-			(font
-				(size 1.27 1.27)
-			)
-			(justify right bottom)
-		)
-	)
 	(label "ROSC"
 		(at 201.93 53.34 180)
@@
 		)
 	)
-	(label "CAN_STB"
-		(at 201.93 63.5 180)
-		(effects
-			(font
-				(size 1.27 1.27)
-			)
-			(justify right bottom)
-		)
-	)
 	(label "RS485_RX"
 		(at 201.93 71.12 180)
@@
 		)
 	)
-	(label "VDDA_EN"
-		(at 201.93 109.22 180)
-		(effects
-			(font
+	(label "ROM_WC"
+		(at 201.93 60.96 180)
+		(effects
+			(font

Commit message: v0.2.9
Parts:
- removed H3: MountingHole, MountingHole:MountingHole_3.2mm_M3_DIN965_Pad, symbol Mechanical:MountingHole
- H1, H2: symbol Mechanical:MountingHole -> Mechanical:MountingHole_Pad
- H3: renamed from H4; symbol Mechanical:MountingHole -> Mechanical:MountingHole_Pad
Connections:
- net GND: now also H1.1, H2.1, H3.1
- net LED1_OUT: now also U1.2 (PA1); no longer U1.1 (PA0_FCC_IN)
- net LED2_OUT: now also U1.1 (PA0_FCC_IN); no longer U1.2 (PA1)
- net SWCLK: now also J1.2 (Pin_2); no longer J1.3 (Pin_3)
- net SWDIO: now also J1.3 (Pin_3); no longer J1.2 (Pin_2)

Commit message: v0.2.10
Parts:
- U2: footprint metis-vela:SO8N_4X5X1P27_STM -> metis-vela:UFDFPN5_1P7X1P4_STM
Connections:
- net +3.3V: now also U2.1 (VCC); no longer U2.8 (VCC)
- net GND: now also U2.2 (VSS); no longer U2.3 (E2), U2.4 (VSS)
- net I2C_SCL: now also U2.4 (SCL); no longer U2.6 (SCL)
- net I2C_SDA: now also U2.3 (SDA); no longer U2.5 (SDA)
- net ROM_WC: now also U2.5 (*WC); no longer U2.7 (*WC)
Changed lines of the file:
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@@
 	(wire
 		(pts
-			(xy 71.12 170.18) (xy 68.58 170.18)
-		)
-		(stroke
-			(width 0)
-			(type default)
-		)
-	)
-	(wire
-		(pts
 			(xy 50.8 40.64) (xy 50.8 43.18)
 		)
@@
 	(wire
 		(pts
-			(xy 68.58 177.8) (xy 68.58 180.34)
+			(xy 68.58 176.53) (xy 68.58 180.34)
 		)
 		(stroke
@@
 	(wire
 		(pts
-			(xy 100.33 175.26) (xy 102.87 175.26)
-		)
-		(stroke
-			(width 0)
-			(type default)
-		)
-	)
-	(wire
-		(pts
 			(xy 201.93 58.42) (xy 207.01 58.42)
 		)
@@
 	(wire
 		(pts
-			(xy 100.33 172.72) (xy 105.41 172.72)
-		)
-		(stroke
-			(width 0)
-			(type default)
-		)
-	)
-	(wire
-		(pts
-			(xy 100.33 170.18) (xy 105.41 170.18)
-		)
-		(stroke
-			(width 0)
-			(type default)
-		)
-	)
-	(wire
-		(pts
-			(xy 100.33 177.8) (xy 105.41 177.8)
+			(xy 57.15 134.62) (xy 57.15 137.16)
 		)
 		(stroke
@@
 	(wire
 		(pts
-			(xy 57.15 134.62) (xy 57.15 137.16)
+			(xy 26.67 124.46) (xy 31.75 124.46)
 		)
 		(stroke
@@
 	(wire
 		(pts
-			(xy 26.67 124.46) (xy 31.75 124.46)
+			(xy 201.93 91.44) (xy 207.01 91.44)
 		)
 		(stroke
@@
 	(wire
 		(pts
-			(xy 201.93 91.44) (xy 207.01 91.44)
+			(xy 201.93 93.98) (xy 207.01 93.98)
 		)
 		(stroke
@@
 	(wire
 		(pts
-			(xy 201.93 93.98) (xy 207.01 93.98)
+			(xy 153.67 35.56) (xy 153.67 43.18)
 		)
 		(stroke
@@
 	(wire
 		(pts
-			(xy 153.67 35.56) (xy 153.67 43.18)
+			(xy 82.55 143.51) (xy 90.17 143.51)
 		)
 		(stroke
@@
 	(wire
 		(pts
-			(xy 82.55 143.51) (xy 90.17 143.51)
+			(xy 99.06 176.53) (xy 104.14 176.53)
 		)
 		(stroke
@@
 	(wire
 		(pts
-			(xy 68.58 167.64) (xy 68.58 170.18)
+			(xy 68.58 167.64) (xy 68.58 171.45)
 		)
 		(stroke
@@
 	(wire
 		(pts
-			(xy 201.93 71.12) (xy 207.01 71.12)
+			(xy 68.58 176.53) (xy 71.12 176.53)
 		)
 		(stroke
@@
 	(wire
 		(pts
-			(xy 39.37 180.34) (xy 39.37 182.88)
+			(xy 201.93 71.12) (xy 207.01 71.12)
 		)
 		(stroke
@@
 	(wire
 		(pts
-			(xy 102.87 175.26) (xy 102.87 180.34)
+			(xy 39.37 180.34) (xy 39.37 182.88)
 		)
 		(stroke
@@
 	(wire
 		(pts
+			(xy 68.58 171.45) (xy 71.12 171.45)
+		)
+		(stroke
+			(width 0)
+			(type default)
+		)
+	)
+	(wire
+		(pts
 			(xy 201.93 114.3) (xy 207.01 114.3)
 		)
@@
 	(wire
 		(pts
-			(xy 71.12 177.8) (xy 68.58 177.8)
-		)
-		(stroke
-			(width 0)
-			(type default)
-		)
-	)
-	(wire
-		(pts
 			(xy 87.63 111.76) (xy 87.63 113.03)
 		)
@@
 	(wire
 		(pts
+			(xy 99.06 171.45) (xy 104.14 171.45)
+		)
+		(stroke
+			(width 0)
+			(type default)
+		)
+	)
+	(wire
+		(pts
 			(xy 62.23 33.02) (xy 62.23 30.48)
 		)
@@
 	(wire
 		(pts
+			(xy 99.06 173.99) (xy 104.14 173.99)
+		)
+		(stroke
+			(width 0)
+			(type default)
+		)
+	)
+	(wire
+		(pts
 			(xy 92.71 35.56) (xy 97.79 35.56)
 		)
@@
 		)
 	)
+	(label "I2C_SCL"
+		(at 104.14 173.99 0)
+		(effects
+			(font
+				(size 1.27 1.27)
+			)
+			(justify left bottom)
+		)
+	)
 	(label "AY_RX"
 		(at 151.13 40.64 180)
@@
 		)
 	)
-	(label "I2C_SCL"
-		(at 105.41 170.18 0)
-		(effects
-			(font
-				(size 1.27 1.27)
-			)
-			(justify left bottom)
-		)
-	)
-	(label "I2C_SDA"
-		(at 105.41 172.72 0)
+	(label "ROM_WC"
+		(at 104.14 171.45 0)
 		(effects
 			(font
@@
 		)
 	)
-	(label "ROM_WC"
-		(at 105.41 177.8 0)
+	(label "RESET"
+		(at 201.93 43.18 180)
 		(effects
 			(font
 				(size 1.27 1.27)
 			)
-			(justify left bottom)
+			(justify right bottom)
 		)
 	)
-	(label "RESET"
-		(at 201.93 43.18 180)
+	(label "VREF-"
+		(at 68.58 85.09 0)
 		(effects
 			(font
 				(size 1.27 1.27)
 			)
-			(justify right bottom)
+			(justify left bottom)
 		)
 	)
-	(label "VREF-"
-		(at 68.58 85.09 0)
+	(label "I2C_SDA"
+		(at 104.14 176.53 0)
 		(effects
 			(font
@@
 	)
 	(symbol
-		(lib_id "Memory_EEPROM:M24C08")
-		(at 71.12 170.18 0)
-		(unit 1)
-		(exclude_from_sim no)
-		(in_bom yes)
-		(on_board yes)
-		(dnp no)
-		(fields_autoplaced yes)
-		(property "Reference" "U2"
-			(at 85.725 162.56 0)
-			(effects
-				(font
-					(size 1.524 1.524)
-				)
-			)
-		)
-		(property "Value" "M24C08"
-			(at 85.725 165.1 0)
-			(effects
-				(font
-					(size 1.524 1.524)
-				)
-			)
-		)
-		(property "Footprint" "metis-vela:SO8N_4X5X1P27_STM"
-			(at 71.12 170.18 0)
-			(effects
-				(font
-					(size 1.27 1.27)
-					(italic yes)
-				)
-				(hide yes)
-			)
-		)
-		(property "Datasheet" "https://www.st.com/resource/en/datasheet/m24c08-r.pdf"
-			(at 71.12 170.18 0)
-			(effects
-				(font
-					(size 1.27 1.27)
-					(italic yes)
-				)
-				(hide yes)
-			)
-		)
-		(property "Description" ""
-			(at 71.12 170.18 0)
-			(effects
-				(font
-					(size 1.27 1.27)
-				)
-				(hide yes)
-			)
-		)
-		(pin "3"
-		)
-		(pin "1"
-		)
-		(pin "4"
-		)
-		(pin "2"
-		)
-		(pin "6"
-		)
-		(pin "8"
-		)
-		(pin "5"
-		)
-		(pin "7"
-		)
-		(instances
-			(project ""
-				(path "/710faa81-ee23-422b-ba7e-b655a364ab6f"
-					(reference "U2")
-					(unit 1)
-				)
-			)
-		)
-	)
-	(symbol
 		(lib_id "power:+3.3V")
 		(at 87.63 111.76 0)
@@
 	)
 	(symbol
-		(lib_id "power:GND")
-		(at 102.87 180.34 0)
-		(unit 1)
-		(exclude_from_sim no)
-		(in_bom yes)
-		(on_board yes)
-		(dnp no)
-		(fields_autoplaced yes)
-		(property "Reference" "#PWR034"
-			(at 102.87 186.69 0)
-			(effects
-				(font
-					(size 1.27 1.27)
-				)
-				(hide yes)
-			)
-		)
-		(property "Value" "GND"
-			(at 102.87 185.42 0)
-			(effects
-				(font
-					(size 1.27 1.27)
-				)
-			)
-		)
-		(property "Footprint" ""
-			(at 102.87 180.34 0)
-			(effects
-				(font
-					(size 1.27 1.27)
-				)
-				(hide yes)
-			)
-		)
-		(property "Datasheet" ""
-			(at 102.87 180.34 0)
-			(effects
-				(font
-					(size 1.27 1.27)
-				)
-				(hide yes)
-			)
-		)
-		(property "Description" "Power symbol creates a global label with name \"GND\" , ground"
-			(at 102.87 180.34 0)
-			(effects
-				(font
-					(size 1.27 1.27)
-				)
-				(hide yes)
-			)
-		)
-		(pin "1"
-		)
-		(instances
-			(project "encoder"
-				(path "/710faa81-ee23-422b-ba7e-b655a364ab6f"
-					(reference "#PWR034")
-					(unit 1)
-				)
-			)
-		)
-	)
-	(symbol
 		(lib_id "power:+3.3V")
 		(at 39.37 170.18 0)
@@
 					(unit 1)
 				)
+			)
+		)
+	)
+	(symbol
+		(lib_id "Memory_EEPROM:M24C08")
+		(at 71.12 171.45 0)
+		(unit 1)
+		(exclude_from_sim no)
+		(in_bom yes)
+		(on_board yes)
+		(dnp no)
+		(fields_autoplaced yes)
+		(property "Reference" "U2"
+			(at 85.09 163.83 0)
+			(effects
+				(font
+					(size 1.524 1.524)
+				)
+			)
+		)
+		(property "Value" "M24C08"
+			(at 85.09 166.37 0)
+			(effects
+				(font
+					(size 1.524 1.524)
+				)
+			)
+		)
+		(property "Footprint" "metis-vela:UFDFPN5_1P7X1P4_STM"
+			(at 71.12 171.45 0)
+			(effects
+				(font
+					(size 1.27 1.27)
+					(italic yes)
+				)
+				(hide yes)
+			)
+		)
+		(property "Datasheet" "https://www.st.com/resource/en/datasheet/m24c08-r.pdf"
+			(at 71.12 171.45 0)
+			(effects
+				(font
+					(size 1.27 1.27)
+					(italic yes)
+				)
+				(hide yes)
+			)
+		)
+		(property "Description" ""
+			(at 71.12 171.45 0)
+			(effects
+				(font
+					(size 1.27 1.27)
+				)
+				(hide yes)
+			)
+		)
+		(pin "2"
+		)
+		(pin "3"
+		)
+		(pin "1"
+		)
+		(pin "4"
+		)
+		(pin "5"
+		)
+		(instances
+			(project ""
+				(path "/710faa81-ee23-422b-ba7e-b655a364ab6f"
+					(reference "U2")
+					(unit 1)
+				)

Commit message: v0.3.0
Parts:
- U1: footprint metis-vela:RHB0032D-IPC_A -> Package_DFN_QFN:Texas_RHB0032E_VQFN-32-1EP_5x5mm_P0.5mm_EP3.45x3.45mm_ThermalVias
Changed lines of the file:
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@@
 			)
 		)
-		(property "Footprint" "metis-vela:RHB0032D-IPC_A"
+		(property "Footprint" "Package_DFN_QFN:Texas_RHB0032E_VQFN-32-1EP_5x5mm_P0.5mm_EP3.45x3.45mm_ThermalVias"
 			(at 207.01 35.56 0)
 			(effects

Commit message: v0.3.2
Parts:
- R5, R6, R8: value 65 -> 150
- R7: value 150 -> 350
Changed lines of the file:
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@@
 			)
 		)
-		(property "Value" "65"
+		(property "Value" "150"
 			(at 82.55 119.38 0)
 			(effects
@@
 			)
 		)
-		(property "Value" "65"
+		(property "Value" "150"
 			(at 135.89 132.08 0)
 			(effects
@@
 			)
 		)
-		(property "Value" "150"
+		(property "Value" "350"
 			(at 124.46 132.08 0)
 			(effects
@@
 			)
 		)
-		(property "Value" "65"
+		(property "Value" "150"
 			(at 92.71 119.38 0)
 			(effects

Commit message: v0.3.5
Parts:
- R7: value 350 -> 348
Changed lines of the file:
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@@
 			)
 		)
-		(property "Value" "350"
+		(property "Value" "348"
 			(at 124.46 132.08 0)
 			(effects
