File: boards/encoder/transmission.kicad_sch (KiCad schematic)
At the start: 32 parts, among them IC1 TPT480, J5 CANbus, J6 RS485, SW4 SW_DPST, U10 TCAN1044V

Commit message: v0.1.14
Parts:
- renumbered C24 to C17, C27 to C18, C28 to C19, C25 to C20, C18 to C21, C21 to C22, C26 to C23, C19 to C24, C22 to C25, C17 to C26, C20 to C27, C23 to C28, D8 to D4, D4 to D5, D9 to D7, D5 to D8, D7 to D9, FL3 to FL1, FL1 to FL2, FL2 to FL3, R26 to R25, R28 to R26, R29 to R27, R25 to R28, R27 to R29, U10 to U8

Commit message: v0.1.15
Parts:
- removed C20, C21, C22, C23, C24, C25: C, symbol Device:C
Other:
- moved on the sheet: D4, D7, FL1, FL2, FL3

Commit message: Added EEPROM
Connections:
- net CAN_H: now also U8.6 (CANL), U8.7 (CANH); no longer FL1.1
- net CAN_L: no longer FL1.3
- net RS485_A: now also IC1.8 (A); no longer FL2.1
- net RS485_B: now also IC1.7 (B); no longer FL2.3
- net RS485_Y: now also IC1.5 (Y); no longer FL3.3
- net RS485_Z: now also IC1.6 (Z); no longer FL3.1
- removed net CAN_H_FILT: FL1.2, FL1.4, U8.6 (CANL), U8.7 (CANH)
- removed net RS485_A_FILT: FL2.2, IC1.8 (A)
- removed net RS485_B_FILT: FL2.4, IC1.7 (B)
- removed net RS485_Y_FILT: FL3.4, IC1.5 (Y)
- removed net RS485_Z_FILT: FL3.2, IC1.6 (Z)
Other:
- moved on the sheet: D4, D6, D7, D9

Commit message: Fixed merge
Parts:
- removed FL1, FL2, FL3: Choke_CommonMode_FerriteCore_1234, symbol Filter:Choke_CommonMode_FerriteCore_1234

Commit message: v0.1.17
Parts:
- removed D4, D5, D6, D7, D8, D9: D_TVS, symbol Device:D_TVS
- added D10, D4, D5: D_TVS_Dual_AAC, Diode_SMD:D_0402_1005Metric, symbol Device:D_TVS_Dual_AAC
Connections:
- net CAN_H: now also D4.1 (A1)
- net CAN_L: now also D4.2 (A2)
- net GND: now also D10.3 (common), D4.3 (common), D5.3 (common)
- net RS485_A: now also D10.1 (A1)
- net RS485_B: now also D10.2 (A2)
- net RS485_Y: now also D5.2 (A2)
- net RS485_Z: now also D5.1 (A1)

Commit message: v0.1.18
Parts:
- renumbered C17 to C13, C18 to C14, C19 to C15, C26 to C16, C27 to C17, C28 to C18, D10 to D4, D4 to D6, J5 to J4, J6 to J5, R24 to R25, R25 to R26, R26 to R27, R27 to R28, R28 to R29, R29 to R30
Other:
- company: (none) -> MetisVela
- title: (none) -> Wanda

Commit message: v0.2.1
Parts:
- C13, C14, C15, C16, C17, C18: footprint (none) -> Capacitor_SMD:C_0603_1608Metric
- R25, R26, R27, R28, R29, R30: footprint (none) -> Resistor_SMD:R_0603_1608Metric
Connections:
- net CAN_H: no longer U8.6 (CANL)
- net CAN_L: now also U8.6 (CANL)
Changed lines of the file:
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@@
 		)
 	)
-	(label "CAN_H_FILT"
+	(label "CAN_L_FILT"
 		(at 74.93 41.91 0)
 		(effects
@@
 			)
 		)
-		(property "Footprint" ""
+		(property "Footprint" "Capacitor_SMD:C_0603_1608Metric"
 			(at 114.3 133.0452 0)
 			(effects
@@
 			)
 		)
-		(property "Footprint" ""
+		(property "Footprint" "Capacitor_SMD:C_0603_1608Metric"
 			(at 171.1452 44.45 0)
 			(effects
@@
 			)
 		)
-		(property "Footprint" ""
+		(property "Footprint" "Resistor_SMD:R_0603_1608Metric"
 			(at 107.95 132.842 90)
 			(effects
@@
 			)
 		)
-		(property "Footprint" ""
+		(property "Footprint" "Resistor_SMD:R_0603_1608Metric"
 			(at 107.95 131.318 90)
 			(effects
@@
 			)
 		)
-		(property "Footprint" ""
+		(property "Footprint" "Resistor_SMD:R_0603_1608Metric"
 			(at 67.818 127 90)
 			(effects
@@
 			)
 		)
-		(property "Footprint" ""
+		(property "Footprint" "Resistor_SMD:R_0603_1608Metric"
 			(at 38.608 127 90)
 			(effects
@@
 			)
 		)
-		(property "Footprint" ""
+		(property "Footprint" "Capacitor_SMD:C_0603_1608Metric"
 			(at 69.85 133.0452 0)
 			(effects
@@
 			)
 		)
-		(property "Footprint" ""
+		(property "Footprint" "Resistor_SMD:R_0603_1608Metric"
 			(at 67.818 137.16 90)
 			(effects
@@
 			)
 		)
-		(property "Footprint" ""
+		(property "Footprint" "Resistor_SMD:R_0603_1608Metric"
 			(at 38.608 137.16 90)
 			(effects
@@
 			)
 		)
-		(property "Footprint" ""
+		(property "Footprint" "Capacitor_SMD:C_0603_1608Metric"
 			(at 183.8452 44.45 0)
 			(effects
@@
 			)
 		)
-		(property "Footprint" ""
+		(property "Footprint" "Capacitor_SMD:C_0603_1608Metric"
 			(at 40.64 133.0452 0)
 			(effects
@@
 			)
 		)
-		(property "Footprint" ""
+		(property "Footprint" "Capacitor_SMD:C_0603_1608Metric"
 			(at 196.5452 44.45 0)
 			(effects
