File: boards/encoder/transmission.kicad_sch (KiCad schematic)
At the start: 20 parts, among them IC1 TPT480, J4 CANbus, J5 RS485, SW4 SW_DPST, U8 TCAN1044V

Commit message: v0.2.2
Parts:
- D4, D5, D6: footprint Diode_SMD:D_0402_1005Metric -> (none)
Changed lines of the file:
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@@
 			)
 		)
-		(property "Footprint" "Diode_SMD:D_0402_1005Metric"
+		(property "Footprint" ""
 			(at 96.52 85.09 0)
 			(effects
@@
 			)
 		)
-		(property "Footprint" "Diode_SMD:D_0402_1005Metric"
+		(property "Footprint" ""
 			(at 67.31 85.09 0)
 			(effects
@@
 			)
 		)
-		(property "Footprint" "Diode_SMD:D_0402_1005Metric"
+		(property "Footprint" ""
 			(at 35.56 85.09 0)
 			(effects

Commit message: Metis-Vela footprint library
Parts:
- IC1: footprint SON65P300X300X80-9N-D -> metis-vela:SON65P300X300X80-9N-D
- U8: footprint SOT-23-THIN-8_DDF_TEX -> metis-vela:SOT-23-THIN-8_DDF_TEX
Changed lines of the file:
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@@
 			)
 		)
-		(property "Footprint" "SON65P300X300X80-9N-D"
+		(property "Footprint" "metis-vela:SON65P300X300X80-9N-D"
 			(at 109.22 127.94 0)
 			(effects
@@
 			)
 		)
-		(property "Footprint" "SOT-23-THIN-8_DDF_TEX"
+		(property "Footprint" "metis-vela:SOT-23-THIN-8_DDF_TEX"
 			(at 33.02 34.29 0)
 			(effects

Commit message: v0.2.3
Parts:
- SW4: value SW_DPST -> 204_211ST; footprint (none) -> metis-vela:SW4_204-211ST_CTS
Connections:
- net CAN_H: now also SW4.1 (3); no longer SW4.3
- net CAN_L: now also SW4.2 (1); no longer SW4.1
- net at R28.1: now also SW4.3 (2); no longer SW4.2
Changed lines of the file:
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@@
 			)
 		)
-		(property "Value" "SW_DPST"
+		(property "Value" "204_211ST"
 			(at 97.79 125.73 0)
 			(effects
@@
 			)
 		)
-		(property "Footprint" ""
+		(property "Footprint" "metis-vela:SW4_204-211ST_CTS"
 			(at 97.79 132.08 0)
 			(effects

Commit message: v0.2.4
Parts:
- D4, D5, D6: footprint (none) -> Package_TO_SOT_SMD:SOT-23-3
Changed lines of the file:
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@@
 			)
 		)
-		(property "Footprint" ""
+		(property "Footprint" "Package_TO_SOT_SMD:SOT-23-3"
 			(at 96.52 85.09 0)
 			(effects
@@
 			)
 		)
-		(property "Footprint" ""
+		(property "Footprint" "Package_TO_SOT_SMD:SOT-23-3"
 			(at 67.31 85.09 0)
 			(effects
@@
 			)
 		)
-		(property "Footprint" ""
+		(property "Footprint" "Package_TO_SOT_SMD:SOT-23-3"
 			(at 35.56 85.09 0)
 			(effects

Commit message: v0.2.7
Connections:
- net RS485_A: no longer D4.1 (A1), IC1.8 (A), R25.1
- net RS485_B: no longer D4.2 (A2), IC1.7 (B), R29.2
- net RS485_Y: no longer D5.2 (A2), IC1.5 (Y), R30.2
- net RS485_Z: no longer D5.1 (A1), IC1.6 (Z), R26.1
- new net RS485_1+: D4.2 (A2), IC1.8 (A), R25.1
- new net RS485_1-: D4.1 (A1), IC1.7 (B), R29.2
- new net RS485_2+: D5.2 (A2), IC1.6 (Z), R26.1
- new net RS485_2-: D5.1 (A1), IC1.5 (Y), R30.2
Changed lines of the file:
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@@
-	)
-	(junction
-		(at 35.56 78.74)
-		(diameter 0)
-		(color 0 0 0 0)
 	)
 	(junction
@@
 	)
 	(junction
-		(at 67.31 99.06)
-		(diameter 0)
-		(color 0 0 0 0)
-	)
-	(junction
-		(at 35.56 99.06)
-		(diameter 0)
-		(color 0 0 0 0)
-	)
-	(junction
-		(at 67.31 78.74)
-		(diameter 0)
-		(color 0 0 0 0)
-	)
-	(junction
 		(at 96.52 99.06)
 		(diameter 0)
@@
 	(wire
 		(pts
-			(xy 35.56 80.01) (xy 35.56 78.74)
-		)
-		(stroke
-			(width 0)
-			(type default)
-		)
-	)
-	(wire
-		(pts
 			(xy 182.88 44.45) (xy 182.88 46.99)
 		)
@@
 	(wire
 		(pts
-			(xy 67.31 78.74) (xy 69.85 78.74)
-		)
-		(stroke
-			(width 0)
-			(type default)
-		)
-	)
-	(wire
-		(pts
 			(xy 62.23 88.9) (xy 62.23 90.17)
 		)
@@
 	(wire
 		(pts
-			(xy 35.56 99.06) (xy 38.1 99.06)
-		)
-		(stroke
-			(width 0)
-			(type default)
-		)
-	)
-	(wire
-		(pts
 			(xy 49.53 132.08) (xy 49.53 133.35)
 		)
@@
 	(wire
 		(pts
-			(xy 38.1 78.74) (xy 35.56 78.74)
-		)
-		(stroke
-			(width 0)
-			(type default)
-		)
-	)
-	(wire
-		(pts
 			(xy 66.04 142.24) (xy 66.04 140.97)
 		)
@@
 	(wire
 		(pts
-			(xy 67.31 99.06) (xy 69.85 99.06)
+			(xy 35.56 78.74) (xy 35.56 80.01)
 		)
 		(stroke
@@
 		)
 	)
-	(label "RS485_Z_FILT"
+	(label "RS485_2+"
 		(at 135.89 43.18 0)
 		(effects
@@
 		)
 	)
-	(label "RS485_Z"
-		(at 64.77 78.74 180)
-		(effects
-			(font
-				(size 1.27 1.27)
-			)
-			(justify right bottom)
-		)
-	)
-	(label "RS485_Z_FILT"
-		(at 69.85 78.74 0)
-		(effects
-			(font
-				(size 1.27 1.27)
-			)
-			(justify left bottom)
-		)
-	)
-	(label "RS485_Z"
-		(at 62.23 121.92 180)
+	(label "RS485_2-"
+		(at 64.77 99.06 180)
 		(effects
 			(font
@@
 		)
 	)
-	(label "RS485_Y"
-		(at 64.77 99.06 180)
-		(effects
-			(font
-				(size 1.27 1.27)
-			)
-			(justify right bottom)
-		)
-	)
-	(label "RS485_A_FILT"
-		(at 38.1 78.74 0)
-		(effects
-			(font
-				(size 1.27 1.27)
-			)
-			(justify left bottom)
-		)
-	)
 	(label "CAN_H_FILT"
 		(at 74.93 39.37 0)
@@
 		)
 	)
-	(label "RS485_Y_FILT"
+	(label "RS485_2-"
 		(at 135.89 45.72 0)
 		(effects
@@
 			)
 			(justify left bottom)
-		)
-	)
-	(label "RS485_B"
-		(at 33.02 142.24 180)
-		(effects
-			(font
-				(size 1.27 1.27)
-			)
-			(justify right bottom)
 		)
 	)
@@
 		)
 	)
+	(label "RS485_1-"
+		(at 33.02 99.06 180)
+		(effects
+			(font
+				(size 1.27 1.27)
+			)
+			(justify right bottom)
+		)
+	)
 	(label "CAN_H"
 		(at 152.4 121.92 180)
@@
 		)
 	)
-	(label "RS485_A"
-		(at 33.02 78.74 180)
+	(label "RS485_2+"
+		(at 64.77 78.74 180)
 		(effects
 			(font
@@
 		)
 	)
-	(label "RS485_Y"
+	(label "RS485_1-"
+		(at 33.02 142.24 180)
+		(effects
+			(font
+				(size 1.27 1.27)
+			)
+			(justify right bottom)
+		)
+	)
+	(label "RS485_1+"
+		(at 135.89 35.56 0)
+		(effects
+			(font
+				(size 1.27 1.27)
+			)
+			(justify left bottom)
+		)
+	)
+	(label "RS485_2-"
 		(at 62.23 142.24 180)
 		(effects
@@
 		)
 	)
-	(label "RS485_Y_FILT"
-		(at 69.85 99.06 0)
-		(effects
-			(font
-				(size 1.27 1.27)
-			)
-			(justify left bottom)
-		)
-	)
-	(label "RS485_A_FILT"
-		(at 135.89 35.56 0)
-		(effects
-			(font
-				(size 1.27 1.27)
-			)
-			(justify left bottom)
-		)
-	)
-	(label "RS485_A"
+	(label "RS485_1+"
 		(at 33.02 121.92 180)
 		(effects
@@
 		)
 	)
-	(label "RS485_B_FILT"
-		(at 38.1 99.06 0)
-		(effects
-			(font
-				(size 1.27 1.27)
-			)
-			(justify left bottom)
-		)
-	)
 	(label "RS485_B"
 		(at 152.4 135.89 180)
@@
 		)
 	)
-	(label "RS485_B_FILT"
+	(label "RS485_1-"
 		(at 135.89 38.1 0)
 		(effects
@@
 		)
 	)
-	(label "RS485_B"
-		(at 33.02 99.06 180)
+	(label "RS485_1+"
+		(at 33.02 78.74 180)
+		(effects
+			(font
+				(size 1.27 1.27)
+			)
+			(justify right bottom)
+		)
+	)
+	(label "RS485_2+"
+		(at 62.23 121.92 180)
 		(effects
 			(font
@@
 		(lib_id "Device:D_TVS_Dual_AAC")
 		(at 67.31 88.9 270)
+		(mirror x)
 		(unit 1)
 		(exclude_from_sim no)
@@
 		(on_board yes)
 		(dnp no)
-		(fields_autoplaced yes)
 		(property "Reference" "D5"
-			(at 69.85 87.6299 90)
+			(at 69.85 90.1701 90)
 			(effects
 				(font
@@
 		)
 		(property "Value" "D_TVS_Dual_AAC"
-			(at 69.85 90.1699 90)
+			(at 69.85 87.6301 90)
 			(effects
 				(font
@@
 		)
 		(property "Footprint" "Package_TO_SOT_SMD:SOT-23-3"
-			(at 67.31 85.09 0)
+			(at 67.31 92.71 0)
 			(effects
 				(font
@@
 		)
 		(property "Datasheet" "~"
-			(at 67.31 85.09 0)
+			(at 67.31 92.71 0)
 			(effects
 				(font
@@
 		(lib_id "Device:D_TVS_Dual_AAC")
 		(at 35.56 88.9 270)
+		(mirror x)
 		(unit 1)
 		(exclude_from_sim no)
@@
 		(on_board yes)
 		(dnp no)
-		(fields_autoplaced yes)
 		(property "Reference" "D4"
-			(at 38.1 87.6299 90)
+			(at 38.1 90.1701 90)
 			(effects
 				(font
@@
 		)
 		(property "Value" "D_TVS_Dual_AAC"
-			(at 38.1 90.1699 90)
+			(at 38.1 87.6301 90)
 			(effects
 				(font
@@
 		)
 		(property "Footprint" "Package_TO_SOT_SMD:SOT-23-3"
-			(at 35.56 85.09 0)
+			(at 35.56 92.71 0)
 			(effects
 				(font
@@
 		)
 		(property "Datasheet" "~"
-			(at 35.56 85.09 0)
-			(effects
-				(font
+			(at 35.56 92.71 0)
+			(effects
+				(font

Commit message: v0.2.8
Parts:
- J5: footprint (none) -> Connector_JST:JST_XH_B4B-XH-A_1x04_P2.50mm_Vertical
Connections:
- net RS485_A is gone; now on net RS485_1+: J5.1 (Pin_1)
- net RS485_B is gone; now on net RS485_1-: J5.2 (Pin_2)
- net RS485_Y is gone; now on net RS485_2-: J5.4 (Pin_4)
- net RS485_Z is gone; now on net RS485_2+: J5.3 (Pin_3)
Changed lines of the file:
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@@
 		)
 	)
-	(label "RS485_Z"
+	(label "RS485_2+"
 		(at 152.4 138.43 180)
 		(effects
@@
 		)
 	)
-	(label "RS485_Y"
+	(label "RS485_2-"
 		(at 152.4 140.97 180)
 		(effects
@@
 		)
 	)
-	(label "RS485_A"
+	(label "RS485_1+"
 		(at 152.4 133.35 180)
 		(effects
@@
 		)
 	)
-	(label "RS485_B"
+	(label "RS485_1-"
 		(at 152.4 135.89 180)
 		(effects
@@
 			)
 		)
-		(property "Footprint" ""
+		(property "Footprint" "Connector_JST:JST_XH_B4B-XH-A_1x04_P2.50mm_Vertical"
 			(at 162.56 135.89 0)
 			(effects

Commit message: v0.2.9
Parts:
- J4: footprint (none) -> Connector_JST:JST_XH_B2B-XH-A_1x02_P2.50mm_Vertical
- renumbered R25 to R23, R26 to R24, R27 to R25, R28 to R26, R29 to R27, R30 to R28, U8 to U9
Connections:
- net CAN_H: now also D6.2 (A2), J4.2 (Pin_2), R25.2; no longer D6.1 (A1), J4.1 (Pin_1), SW4.1 (3)
- net CAN_L: now also D6.1 (A1), J4.1 (Pin_1), R26.1; no longer D6.2 (A2), J4.2 (Pin_2), SW4.2 (1)
- net at SW4.3 (2): now also C18.2, SW4.4; no longer R26.1
- new net: R26.2, SW4.2 (1)
- new net: R25.1, SW4.1 (3)
Other:
- moved on the sheet: R25, R26, SW4

Commit message: v0.3.0
Changed lines of the file:
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@@
-	)
-	(junction
-		(at 96.52 78.74)
-		(diameter 0)
-		(color 0 0 0 0)
 	)
 	(junction
@@
 		(color 0 0 0 0)
 	)
-	(junction
-		(at 96.52 99.06)
-		(diameter 0)
-		(color 0 0 0 0)
-	)
 	(wire
 		(pts
@@
 	(wire
 		(pts
-			(xy 96.52 78.74) (xy 99.06 78.74)
-		)
-		(stroke
-			(width 0)
-			(type default)
-		)
-	)
-	(wire
-		(pts
 			(xy 69.85 39.37) (xy 74.93 39.37)
 		)
@@
 		(pts
 			(xy 36.83 142.24) (xy 36.83 140.97)
-		)
-		(stroke
-			(width 0)
-			(type default)
-		)
-	)
-	(wire
-		(pts
-			(xy 96.52 99.06) (xy 99.06 99.06)
 		)
 		(stroke
@@
 		)
 	)
-	(label "CAN_L_FILT"
-		(at 99.06 99.06 0)
-		(effects
-			(font
-				(size 1.27 1.27)
-			)
-			(justify left bottom)
-		)
-	)
-	(label "CAN_H_FILT"
+	(label "CAN_H"
 		(at 74.93 39.37 0)
 		(effects
@@
 		)
 	)
-	(label "CAN_L_FILT"
+	(label "CAN_L"
 		(at 74.93 41.91 0)
 		(effects
@@
 		)
 	)
-	(label "CAN_H_FILT"
-		(at 99.0339 78.74 0)
-		(effects
-			(font
-				(size 1.27 1.27)
-			)
-			(justify left bottom)
-		)
-	)
