File: boards/encoder/transmission.kicad_sch (KiCad schematic)
At the start: 20 parts, among them IC1 TPT480, J4 CANbus, J5 RS485, SW4 204_211ST, U9 TCAN1044V

Commit message: v0.3.10
Parts:
- R21: renamed from R23; value 60 -> 60.4
- R22: renamed from R24; value 60 -> 60.4
- R23: renamed from R25; value 60 -> 60.4
- R24: renamed from R26; value 60 -> 60.4
- R25: renamed from R27; value 60 -> 60.4
- R26: renamed from R28; value 60 -> 60.4
Changed lines of the file:
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@@
+			)
+		)
+		(property "Sim.Type" ""
+			(at 118.11 132.08 90)
+			(effects
+				(font
+					(size 1.27 1.27)
+				)
+				(hide yes)
 			)
 		)
@@
 			)
 		)
+		(property "Sim.Type" ""
+			(at 170.18 40.64 0)
+			(effects
+				(font
+					(size 1.27 1.27)
+				)
+				(hide yes)
+			)
+		)
 		(pin "1"
 		)
@@
 			)
 		)
+		(property "Sim.Type" ""
+			(at 96.52 88.9 90)
+			(effects
+				(font
+					(size 1.27 1.27)
+				)
+				(hide yes)
+			)
+		)
 		(pin "3"
 		)
@@
 			)
 		)
+		(property "Sim.Type" ""
+			(at 130.81 33.02 0)
+			(effects
+				(font
+					(size 1.27 1.27)
+				)
+				(hide yes)
+			)
+		)
 		(pin "6"
 		)
@@
 		(on_board yes)
 		(dnp no)
-		(property "Reference" "R26"
+		(property "Reference" "R24"
 			(at 94.488 137.922 90)
 			(effects
@@
 			)
 		)
-		(property "Value" "60"
+		(property "Value" "60.4"
 			(at 94.488 140.462 90)
 			(effects
@@
 			)
 		)
+		(property "Sim.Type" ""
+			(at 96.52 134.62 90)
+			(effects
+				(font
+					(size 1.27 1.27)
+				)
+				(hide yes)
+			)
+		)
 		(pin "1"
 		)
@@
 			(project "encoder"
 				(path "/710faa81-ee23-422b-ba7e-b655a364ab6f/7d4fde09-a0e3-44c6-b789-9c20af482bf4"
-					(reference "R26")
+					(reference "R24")
 					(unit 1)
 				)
@@
 			)
 		)
+		(property "Sim.Type" ""
+			(at 162.56 135.89 0)
+			(effects
+				(font
+					(size 1.27 1.27)
+				)
+				(hide yes)
+			)
+		)
 		(pin "3"
 		)
@@
 		(on_board yes)
 		(dnp no)
-		(property "Reference" "R25"
+		(property "Reference" "R23"
 			(at 94.996 123.952 90)
 			(effects
@@
 			)
 		)
-		(property "Value" "60"
+		(property "Value" "60.4"
 			(at 94.996 126.492 90)
 			(effects
@@
 			)
 		)
+		(property "Sim.Type" ""
+			(at 96.52 129.54 90)
+			(effects
+				(font
+					(size 1.27 1.27)
+				)
+				(hide yes)
+			)
+		)
 		(pin "1"
 		)
@@
 			(project "encoder"
 				(path "/710faa81-ee23-422b-ba7e-b655a364ab6f/7d4fde09-a0e3-44c6-b789-9c20af482bf4"
-					(reference "R25")
+					(reference "R23")
 					(unit 1)
 				)
@@
 			)
 		)
+		(property "Sim.Type" ""
+			(at 67.31 88.9 90)
+			(effects
+				(font
+					(size 1.27 1.27)
+				)
+				(hide yes)
+			)
+		)
 		(pin "3"
 		)
@@
 		(on_board yes)
 		(dnp no)
-		(property "Reference" "R24"
+		(property "Reference" "R22"
 			(at 63.5 125.7299 0)
 			(effects
@@
 			)
 		)
-		(property "Value" "60"
+		(property "Value" "60.4"
 			(at 63.5 128.2699 0)
 			(effects
@@
 			)
 		)
+		(property "Sim.Type" ""
+			(at 66.04 127 0)
+			(effects
+				(font
+					(size 1.27 1.27)
+				)
+				(hide yes)
+			)
+		)
 		(pin "1"
 		)
@@
 			(project "encoder"
 				(path "/710faa81-ee23-422b-ba7e-b655a364ab6f/7d4fde09-a0e3-44c6-b789-9c20af482bf4"
-					(reference "R24")
+					(reference "R22")
 					(unit 1)
 				)
@@
 		(on_board yes)
 		(dnp no)
-		(property "Reference" "R23"
+		(property "Reference" "R21"
 			(at 34.29 125.7299 0)
 			(effects
@@
 			)
 		)
-		(property "Value" "60"
+		(property "Value" "60.4"
 			(at 34.29 128.2699 0)
 			(effects
@@
 			)
 		)
+		(property "Sim.Type" ""
+			(at 36.83 127 0)
+			(effects
+				(font
+					(size 1.27 1.27)
+				)
+				(hide yes)
+			)
+		)
 		(pin "1"
 		)
@@
 			(project "encoder"
 				(path "/710faa81-ee23-422b-ba7e-b655a364ab6f/7d4fde09-a0e3-44c6-b789-9c20af482bf4"
-					(reference "R23")
+					(reference "R21")
 					(unit 1)
 				)
@@
 			)
 		)
+		(property "Sim.Type" ""
+			(at 73.66 132.08 90)
+			(effects
+				(font
+					(size 1.27 1.27)
+				)
+				(hide yes)
+			)
+		)
 		(pin "1"
 		)
@@
 			)
 		)
+		(property "Sim.Type" ""
+			(at 33.02 34.29 0)
+			(effects
+				(font
+					(size 1.27 1.27)
+				)
+				(hide yes)
+			)
+		)
 		(pin "4"
 		)
@@
 			)
 		)
+		(property "Sim.Type" ""
+			(at 35.56 88.9 90)
+			(effects
+				(font
+					(size 1.27 1.27)
+				)
+				(hide yes)
+			)
+		)
 		(pin "3"
 		)
@@
 		(on_board yes)
 		(dnp no)
-		(property "Reference" "R28"
+		(property "Reference" "R26"
 			(at 63.5 135.8899 0)
 			(effects
@@
 			)
 		)
-		(property "Value" "60"
+		(property "Value" "60.4"
 			(at 63.5 138.4299 0)
 			(effects
@@
 			)
 		)
+		(property "Sim.Type" ""
+			(at 66.04 137.16 0)
+			(effects
+				(font
+					(size 1.27 1.27)
+				)
+				(hide yes)
+			)
+		)
 		(pin "1"
 		)
@@
 			(project "encoder"
 				(path "/710faa81-ee23-422b-ba7e-b655a364ab6f/7d4fde09-a0e3-44c6-b789-9c20af482bf4"
-					(reference "R28")
+					(reference "R26")
 					(unit 1)
 				)
@@
 			)
 		)
+		(property "Sim.Type" ""
+			(at 162.56 121.92 0)
+			(effects
+				(font
+					(size 1.27 1.27)
+				)
+				(hide yes)
+			)
+		)
 		(pin "2"
 		)
@@
 		(on_board yes)
 		(dnp no)
-		(property "Reference" "R27"
+		(property "Reference" "R25"
 			(at 34.29 135.8899 0)
 			(effects
@@
 			)
 		)
-		(property "Value" "60"
+		(property "Value" "60.4"
 			(at 34.29 138.4299 0)
 			(effects
@@
 			)
 		)
+		(property "Sim.Type" ""
+			(at 36.83 137.16 0)
+			(effects
+				(font
+					(size 1.27 1.27)
+				)
+				(hide yes)
+			)
+		)
 		(pin "1"
 		)
@@
 			(project "encoder"
 				(path "/710faa81-ee23-422b-ba7e-b655a364ab6f/7d4fde09-a0e3-44c6-b789-9c20af482bf4"
-					(reference "R27")
+					(reference "R25")
 					(unit 1)
 				)
@@
 			)
 		)
+		(property "Sim.Type" ""
+			(at 182.88 40.64 0)
+			(effects
+				(font
+					(size 1.27 1.27)
+				)
+				(hide yes)
+			)
+		)
 		(pin "1"
 		)
@@
 			)
 		)
+		(property "Sim.Type" ""
+			(at 44.45 132.08 90)
+			(effects
+				(font
+					(size 1.27 1.27)
+				)
+				(hide yes)
+			)
+		)
 		(pin "1"
 		)
@@
 			)
 		)
+		(property "Sim.Type" ""
+			(at 106.68 132.08 0)
+			(effects
+				(font
+					(size 1.27 1.27)
+				)
+				(hide yes)
+			)
+		)
 		(pin "3"
 		)
@@
 			(at 195.58 40.64 0)
 			(effects
+				(font
+					(size 1.27 1.27)
+				)
+				(hide yes)
+			)
+		)
+		(property "Sim.Type" ""
+			(at 195.58 40.64 0)
+			(effects
