File: boards/encoder/analog.kicad_sch (KiCad schematic)
At the start: 29 parts, among them Q1 NPN, Q2 PNP, Q3 NMOS, U3 AZ431-A, U4 CT310, U5 Opamp_Dual, U7 INA826, U9 INA826

Commit message: v0.1.14
Parts:
- removed Q1: NPN, symbol Simulation_SPICE:NPN
- removed Q2: PNP, symbol Simulation_SPICE:PNP
- added Q1: QSZ2TR, symbol Transistor_BJT:Q_Dual_NPN_PNP_B1E2B2C2E1C1
- C10: renamed from C16; value C -> 5600p
- C9: renamed from C15; value C -> 5600p
- R11: renamed from R22; value R -> 470
- R12: renamed from R23; value R -> 470
- R13: renamed from R18; value R -> 60.4k
- R14: renamed from R20; value R -> 60.4k
- renumbered C9 to C11, C10 to C12, C11 to C13, C12 to C14, C13 to C15, C14 to C16, Q3 to Q2, R11 to R15, R15 to R16, R12 to R17, R19 to R18, R16 to R19, R13 to R20, R17 to R21, R21 to R22, R14 to R23, U4 to U3, U7 to U4, U9 to U5, U5 to U6, U3 to U7
Connections:
- net GND: now also Q1.2 (E2)
- net VBIAS: now also Q1.4 (C2), Q1.5 (E1)
- net VDDA: now also Q1.6 (C1)
- net at R18.2: now also Q1.1 (B1), Q1.3 (B2)
Other:
- moved on the sheet: C14, C15, C16

Commit message: v0.1.16
Parts:
- removed Q2: NMOS, symbol Simulation_SPICE:NMOS
- added Q2: PMOS, symbol Simulation_SPICE:PMOS
- R13, R14: value 60.4k -> 98.8k
Connections:
- net GND: no longer R22.1
- net VDD: now also R22.1, Q2.3 (S)
- net VDDA: now also Q2.1 (D)
- net VDDA_EN: now also Q2.2 (G)

Commit message: v0.1.17
Other:
- moved on the sheet: Q2, R22
Changed lines of the file:
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@@
 	)
 	(junction
-		(at 209.55 101.6)
-		(diameter 0)
-		(color 0 0 0 0)
-	)
-	(junction
 		(at 72.39 96.52)
 		(diameter 0)
@@
 	)
 	(junction
-		(at 45.72 86.36)
+		(at 199.39 97.79)
 		(diameter 0)
 		(color 0 0 0 0)
 	)
 	(junction
-		(at 196.85 91.44)
+		(at 45.72 86.36)
 		(diameter 0)
 		(color 0 0 0 0)
@@
 		(color 0 0 0 0)
 	)
+	(junction
+		(at 199.39 86.36)
+		(diameter 0)
+		(color 0 0 0 0)
+	)
 	(wire
 		(pts
-			(xy 215.9 81.28) (xy 215.9 91.44)
+			(xy 207.01 93.98) (xy 207.01 97.79)
+		)
+		(stroke
+			(width 0)
+			(type default)
+		)
+	)
+	(wire
+		(pts
+			(xy 199.39 97.79) (xy 199.39 96.52)
+		)
+		(stroke
+			(width 0)
+			(type default)
+		)
+	)
+	(wire
+		(pts
+			(xy 214.63 83.82) (xy 214.63 86.36)
 		)
 		(stroke
@@
 	(wire
 		(pts
-			(xy 196.85 91.44) (xy 196.85 93.98)
+			(xy 199.39 86.36) (xy 199.39 88.9)
 		)
 		(stroke
@@
 	(wire
 		(pts
-			(xy 214.63 91.44) (xy 215.9 91.44)
+			(xy 212.09 86.36) (xy 214.63 86.36)
 		)
 		(stroke
@@
 	(wire
 		(pts
-			(xy 196.85 91.44) (xy 191.77 91.44)
+			(xy 199.39 97.79) (xy 207.01 97.79)
 		)
 		(stroke
@@
 	(wire
 		(pts
+			(xy 199.39 86.36) (xy 196.85 86.36)
+		)
+		(stroke
+			(width 0)
+			(type default)
+		)
+	)
+	(wire
+		(pts
 			(xy 106.68 92.71) (xy 106.68 93.98)
 		)
@@
 	(wire
 		(pts
-			(xy 191.77 91.44) (xy 191.77 81.28)
-		)
-		(stroke
-			(width 0)
-			(type default)
-		)
-	)
-	(wire
-		(pts
 			(xy 181.61 35.56) (xy 181.61 36.83)
 		)
@@
 	(wire
 		(pts
-			(xy 209.55 101.6) (xy 196.85 101.6)
-		)
-		(stroke
-			(width 0)
-			(type default)
-		)
-	)
-	(wire
-		(pts
 			(xy 29.21 39.37) (xy 34.29 39.37)
 		)
@@
 	(wire
 		(pts
+			(xy 196.85 86.36) (xy 196.85 83.82)
+		)
+		(stroke
+			(width 0)
+			(type default)
+		)
+	)
+	(wire
+		(pts
 			(xy 45.72 87.63) (xy 45.72 86.36)
 		)
@@
 	(wire
 		(pts
-			(xy 209.55 107.95) (xy 209.55 101.6)
-		)
-		(stroke
-			(width 0)
-			(type default)
-		)
-	)
-	(wire
-		(pts
-			(xy 204.47 91.44) (xy 196.85 91.44)
-		)
-		(stroke
-			(width 0)
-			(type default)
-		)
-	)
-	(wire
-		(pts
-			(xy 209.55 99.06) (xy 209.55 101.6)
+			(xy 199.39 104.14) (xy 199.39 97.79)
 		)
 		(stroke
@@
 	(wire
 		(pts
-			(xy 191.77 107.95) (xy 209.55 107.95)
+			(xy 196.85 104.14) (xy 199.39 104.14)
 		)
 		(stroke
@@
 	(wire
 		(pts
+			(xy 199.39 86.36) (xy 201.93 86.36)
+		)
+		(stroke
+			(width 0)
+			(type default)
+		)
+	)
+	(wire
+		(pts
 			(xy 31.75 139.7) (xy 31.75 142.24)
 		)
@@
 	(hierarchical_label "VDDA_EN"
 		(shape input)
-		(at 191.77 107.95 180)
+		(at 196.85 104.14 180)
 		(effects
 			(font
@@
 	(symbol
 		(lib_id "power:VDD")
-		(at 191.77 81.28 0)
+		(at 196.85 83.82 0)
 		(unit 1)
 		(exclude_from_sim no)
@@
 		(fields_autoplaced yes)
 		(property "Reference" "#PWR050"
-			(at 191.77 85.09 0)
+			(at 196.85 87.63 0)
 			(effects
 				(font
@@
 		)
 		(property "Value" "VDD"
-			(at 191.77 76.2 0)
+			(at 196.85 78.74 0)
 			(effects
 				(font
@@
 		)
 		(property "Footprint" ""
-			(at 191.77 81.28 0)
+			(at 196.85 83.82 0)
 			(effects
 				(font
@@
 		)
 		(property "Datasheet" ""
-			(at 191.77 81.28 0)
+			(at 196.85 83.82 0)
 			(effects
 				(font
@@
 		)
 		(property "Description" "Power symbol creates a global label with name \"VDD\""
-			(at 191.77 81.28 0)
+			(at 196.85 83.82 0)
 			(effects
 				(font
@@
 	(symbol
 		(lib_id "Device:R")
-		(at 196.85 97.79 0)
+		(at 199.39 92.71 0)
 		(unit 1)
 		(exclude_from_sim no)
@@
 		(fields_autoplaced yes)
 		(property "Reference" "R22"
-			(at 199.39 96.5199 0)
+			(at 201.93 91.4399 0)
 			(effects
 				(font
@@
 		)
 		(property "Value" "R"
-			(at 199.39 99.0599 0)
+			(at 201.93 93.9799 0)
 			(effects
 				(font
@@
 		)
 		(property "Footprint" ""
-			(at 195.072 97.79 90)
+			(at 197.612 92.71 90)
 			(effects
 				(font
@@
 		)
 		(property "Datasheet" "~"
-			(at 196.85 97.79 0)
+			(at 199.39 92.71 0)
 			(effects
 				(font
@@
 		)
 		(property "Description" "Resistor"
-			(at 196.85 97.79 0)
+			(at 199.39 92.71 0)
 			(effects
 				(font
@@
 	(symbol
 		(lib_id "power:VDDA")
-		(at 215.9 81.28 0)
+		(at 214.63 83.82 0)
 		(unit 1)
 		(exclude_from_sim no)
@@
 		(fields_autoplaced yes)
 		(property "Reference" "#PWR051"
-			(at 215.9 85.09 0)
+			(at 214.63 87.63 0)
 			(effects
 				(font
@@
 		)
 		(property "Value" "VDDA"
-			(at 215.9 76.2 0)
+			(at 214.63 78.74 0)
 			(effects
 				(font
@@
 		)
 		(property "Footprint" ""
-			(at 215.9 81.28 0)
+			(at 214.63 83.82 0)
 			(effects
 				(font
@@
 		)
 		(property "Datasheet" ""
-			(at 215.9 81.28 0)
+			(at 214.63 83.82 0)
 			(effects
 				(font
@@
 		)
 		(property "Description" "Power symbol creates a global label with name \"VDDA\""
-			(at 215.9 81.28 0)
+			(at 214.63 83.82 0)
 			(effects
 				(font
@@
 	(symbol
 		(lib_id "Simulation_SPICE:PMOS")
-		(at 209.55 93.98 270)
+		(at 207.01 88.9 270)
 		(mirror x)
 		(unit 1)
@@
 		(dnp no)
 		(property "Reference" "Q2"
-			(at 211.074 87.376 0)
+			(at 208.534 82.296 0)
 			(effects
 				(font
@@
 		)
 		(property "Value" "PMOS"
-			(at 208.534 87.376 0)
+			(at 205.994 82.296 0)
 			(effects
 				(font
@@
 		)
 		(property "Footprint" ""
-			(at 212.09 88.9 0)
+			(at 209.55 83.82 0)
 			(effects
 				(font
@@
 		)
 		(property "Datasheet" "https://ngspice.sourceforge.io/docs/ngspice-html-manual/manual.xhtml#cha_MOSFETs"
-			(at 196.85 93.98 0)
+			(at 194.31 88.9 0)
 			(effects
 				(font
@@
 		)
 		(property "Description" "P-MOSFET transistor, drain/source/gate"
-			(at 209.55 93.98 0)
+			(at 207.01 88.9 0)
 			(effects
 				(font
@@
 		)
 		(property "Sim.Device" "PMOS"
-			(at 192.405 93.98 0)
+			(at 189.865 88.9 0)
 			(effects
 				(font
@@
 		)
 		(property "Sim.Type" "VDMOS"
-			(at 190.5 93.98 0)
+			(at 187.96 88.9 0)
 			(effects
 				(font
@@
 		)
 		(property "Sim.Pins" "1=D 2=G 3=S"
-			(at 194.31 93.98 0)
+			(at 191.77 88.9 0)
 			(effects
 				(font

Commit message: v0.1.18
Parts:
- renumbered C14 to C10, C15 to C11, C16 to C12, C9 to C5, C10 to C6, C11 to C7, C12 to C8, C13 to C9, R11 to R12, R12 to R13, R13 to R14, R14 to R15, R15 to R16, R16 to R17, R17 to R18, R18 to R19, R22 to R20, R19 to R21, R20 to R22, R21 to R23, R23 to R24
Other:
- company: (none) -> MetisVela
- title: (none) -> Wanda

Commit message: v0.1.19
Parts:
- C10, C11, C12: value C -> 100n
- C7: value C -> 1u
- C8, C9: value C -> 10u
- R16, R18, R24: value R -> 20k
- R17, R21: value R -> 10k
- R19, R23: value R -> 9.8k
- R22: value R -> 100k
Changed lines of the file:
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@@
 			)
 		)
-		(property "Value" "R"
+		(property "Value" "10k"
 			(at 109.22 90.1699 0)
 			(effects
@@
 			)
 		)
-		(property "Value" "C"
+		(property "Value" "10u"
 			(at 66.04 147.3199 0)
 			(effects
@@
 			)
 		)
-		(property "Value" "C"
+		(property "Value" "1u"
 			(at 35.56 147.3199 0)
 			(effects
@@
 			)
 		)
-		(property "Value" "C"
+		(property "Value" "100n"
 			(at 116.84 147.3199 0)
 			(effects
@@
 			)
 		)
-		(property "Value" "R"
+		(property "Value" "20k"
 			(at 48.26 92.7099 0)
 			(effects
@@
 			)
 		)
-		(property "Value" "R"
+		(property "Value" "10k"
 			(at 109.22 100.3299 0)
 			(effects
@@
 			)
 		)
-		(property "Value" "C"
+		(property "Value" "100n"
 			(at 93.98 147.3199 0)
 			(effects
@@
 			)
 		)
-		(property "Value" "R"
+		(property "Value" "20k"
 			(at 64.77 102.87 90)
 			(effects
@@
 			)
 		)
-		(property "Value" "R"
+		(property "Value" "100k"
 			(at 48.26 102.8699 0)
 			(effects
@@
 			)
 		)
-		(property "Value" "R"
+		(property "Value" "9.8k"
 			(at 119.38 107.95 90)
 			(effects
@@
 			)
 		)
-		(property "Value" "C"
+		(property "Value" "10u"
 			(at 54.61 147.3199 0)
 			(effects
@@
 			)
 		)
-		(property "Value" "R"
+		(property "Value" "9.8k"
 			(at 135.89 88.9 90)
 			(effects
@@
 			)
 		)
-		(property "Value" "R"
+		(property "Value" "20k"
 			(at 33.02 82.55 90)
 			(effects
@@
 			)
 		)
-		(property "Value" "C"
+		(property "Value" "100n"
 			(at 105.41 147.3199 0)
 			(effects

Commit message: Fixed some values
Parts:
- C8, C9: value 10u -> 1u
- R16, R24: value 20k -> 100
- R18: value 20k -> 10k
- R19, R23: value 9.8k -> 100
- R20: value R -> 10k
- R22: value 100k -> 50k
Changed lines of the file:
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@@
 			)
 		)
-		(property "Value" "10u"
+		(property "Value" "1u"
 			(at 66.04 147.3199 0)
 			(effects
@@
 			)
 		)
-		(property "Value" "20k"
+		(property "Value" "10k"
 			(at 48.26 92.7099 0)
 			(effects
@@
 			)
 		)
-		(property "Value" "20k"
+		(property "Value" "100"
 			(at 64.77 102.87 90)
 			(effects
@@
 			)
 		)
-		(property "Value" "100k"
+		(property "Value" "50k"
 			(at 48.26 102.8699 0)
 			(effects
@@
 			)
 		)
-		(property "Value" "9.8k"
+		(property "Value" "100"
 			(at 119.38 107.95 90)
 			(effects
@@
 			)
 		)
-		(property "Value" "10u"
+		(property "Value" "1u"
 			(at 54.61 147.3199 0)
 			(effects
@@
 			)
 		)
-		(property "Value" "9.8k"
+		(property "Value" "100"
 			(at 135.89 88.9 90)
 			(effects
@@
 			)
 		)
-		(property "Value" "R"
+		(property "Value" "10k"
 			(at 201.93 93.9799 0)
 			(effects
@@
 			)
 		)
-		(property "Value" "20k"
+		(property "Value" "100"
 			(at 33.02 82.55 90)
 			(effects

Commit message: v0.2.1
Parts:
- C10, C11, C12, C5, C6, C7, C8, C9: footprint (none) -> Capacitor_SMD:C_0603_1608Metric
- R12, R13, R14, R15, R16, R17, R18, R19, R20, R21, R22, R23, R24: footprint (none) -> Resistor_SMD:R_0603_1608Metric
- U3: footprint (none) -> Package_DFN_QFN:DFN-8-1EP_2x2mm_P0.5mm_EP0.8x1.6mm
- U4, U5: footprint INA826AIDRGR:SON50P300X300X80-9N200X120 -> Package_SON:SON50P300X300X80-9N200X120
Connections:
- net GND: now also U3.9 (EP)
- net at R18.1, R22.2: now also U7.1 (REF); no longer U7.2 (REF)
- net at R16.2, R18.2, U6.3 (+): now also U7.2 (K); no longer U7.1 (K)
Changed lines of the file:
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@@
 	(wire
 		(pts
+			(xy 45.72 50.8) (xy 45.72 49.53)
+		)
+		(stroke
+			(width 0)
+			(type default)
+		)
+	)
+	(wire
+		(pts
 			(xy 114.3 101.6) (xy 114.3 95.25)
 		)
@@
 			)
 		)
-		(property "Footprint" ""
+		(property "Footprint" "Resistor_SMD:R_0603_1608Metric"
 			(at 104.902 88.9 90)
 			(effects
@@
 			)
 		)
-		(property "Footprint" ""
+		(property "Footprint" "Capacitor_SMD:C_0603_1608Metric"
 			(at 61.2648 142.24 0)
 			(effects
@@
 	(symbol
 		(lib_id "power:GNDA")
+		(at 45.72 50.8 0)
+		(unit 1)
+		(exclude_from_sim no)
+		(in_bom yes)
+		(on_board yes)
+		(dnp no)
+		(fields_autoplaced yes)
+		(property "Reference" "#PWR092"
+			(at 45.72 57.15 0)
+			(effects
+				(font
+					(size 1.27 1.27)
+				)
+				(hide yes)
+			)
+		)
+		(property "Value" "GNDA"
+			(at 45.72 55.88 0)
+			(effects
+				(font
+					(size 1.27 1.27)
+				)
+			)
+		)
+		(property "Footprint" ""
+			(at 45.72 50.8 0)
+			(effects
+				(font
+					(size 1.27 1.27)
+				)
+				(hide yes)
+			)
+		)
+		(property "Datasheet" ""
+			(at 45.72 50.8 0)
+			(effects
+				(font
+					(size 1.27 1.27)
+				)
+				(hide yes)
+			)
+		)
+		(property "Description" "Power symbol creates a global label with name \"GNDA\" , analog ground"
+			(at 45.72 50.8 0)
+			(effects
+				(font
+					(size 1.27 1.27)
+				)
+				(hide yes)
+			)
+		)
+		(pin "1"
+		)
+		(instances
+			(project "encoder"
+				(path "/710faa81-ee23-422b-ba7e-b655a364ab6f/763a463a-636e-4b92-a93e-dd97da54b348"
+					(reference "#PWR092")
+					(unit 1)
+				)
+			)
+		)
+	)
+	(symbol
+		(lib_id "power:GNDA")
 		(at 127 49.53 0)
 		(unit 1)
@@
 			)
 		)
-		(property "Footprint" ""
+		(property "Footprint" "Capacitor_SMD:C_0603_1608Metric"
 			(at 32.7152 149.86 0)
 			(effects
@@
 			)
 		)
-		(property "Footprint" ""
+		(property "Footprint" "Capacitor_SMD:C_0603_1608Metric"
 			(at 113.9952 149.86 0)
 			(effects
@@
 			)
 		)
-		(property "Footprint" ""
+		(property "Footprint" "Resistor_SMD:R_0603_1608Metric"
 			(at 47.498 91.44 90)
 			(effects
@@
 			)
 		)
-		(property "Footprint" ""
+		(property "Footprint" "Resistor_SMD:R_0603_1608Metric"
 			(at 108.458 99.06 90)
 			(effects
@@
 			)
 		)
-		(property "Footprint" ""
+		(property "Footprint" "Capacitor_SMD:C_0603_1608Metric"
 			(at 91.1352 149.86 0)
 			(effects
@@
 			)
 		)
-		(property "Footprint" ""
+		(property "Footprint" "Resistor_SMD:R_0603_1608Metric"
 			(at 64.77 108.458 90)
 			(effects
@@
 			)
 		)
-		(property "Footprint" ""
+		(property "Footprint" "Resistor_SMD:R_0603_1608Metric"
 			(at 47.498 101.6 90)
 			(effects
@@
 			)
 		)
-		(property "Footprint" "INA826AIDRGR:SON50P300X300X80-9N200X120"
+		(property "Footprint" "Package_SON:SON50P300X300X80-9N200X120"
 			(at 109.22 41.91 0)
 			(effects
@@
 			)
 		)
-		(property "Footprint" ""
+		(property "Footprint" "Resistor_SMD:R_0603_1608Metric"
 			(at 119.38 99.822 90)
 			(effects
@@
 			)
 		)
-		(property "Footprint" ""
+		(property "Footprint" "Capacitor_SMD:C_0603_1608Metric"
 			(at 214.3252 49.53 0)
 			(effects
@@
 			)
 		)
-		(property "Footprint" ""
+		(property "Footprint" "Capacitor_SMD:C_0603_1608Metric"
 			(at 49.8348 142.24 0)
 			(effects
@@
 			)
 		)
-		(property "Footprint" ""
+		(property "Footprint" "Resistor_SMD:R_0603_1608Metric"
 			(at 135.89 94.488 90)
 			(effects
@@
 			)
 		)
-		(property "Footprint" ""
+		(property "Footprint" "Resistor_SMD:R_0603_1608Metric"
 			(at 211.582 35.56 90)
 			(effects
@@
 			)
 		)
-		(property "Footprint" ""
+		(property "Footprint" "Resistor_SMD:R_0603_1608Metric"
 			(at 126.492 40.64 90)
 			(effects
@@
 			)
 		)
-		(property "Footprint" ""
+		(property "Footprint" "Resistor_SMD:R_0603_1608Metric"
 			(at 179.832 40.64 90)
 			(effects
@@
 			)
 		)
-		(property "Footprint" ""
+		(property "Footprint" "Resistor_SMD:R_0603_1608Metric"
 			(at 197.612 92.71 90)
 			(effects
@@
 			)
 		)
-		(property "Footprint" ""
+		(property "Footprint" "Package_DFN_QFN:DFN-8-1EP_2x2mm_P0.5mm_EP0.8x1.6mm"
 			(at 45.72 40.64 0)
 			(effects
@@
 		(pin "1"
 		)
+		(pin "9"
+		)
 		(instances
 			(project "analog"
@@
 			)
 		)
-		(property "Footprint" ""
+		(property "Footprint" "Capacitor_SMD:C_0603_1608Metric"
 			(at 229.5652 49.53 0)
 			(effects
@@
 			)
 		)
-		(property "Footprint" "INA826AIDRGR:SON50P300X300X80-9N200X120"
+		(property "Footprint" "Package_SON:SON50P300X300X80-9N200X120"
 			(at 162.56 41.91 0)
 			(effects
@@
 			)
 		)
-		(property "Footprint" ""
+		(property "Footprint" "Resistor_SMD:R_0603_1608Metric"
 			(at 33.02 88.138 90)
 			(effects
@@
 			)
 		)
-		(property "Footprint" ""
+		(property "Footprint" "Resistor_SMD:R_0603_1608Metric"
 			(at 226.822 35.56 90)
 			(effects
@@
 			)
 		)
-		(property "Footprint" ""
+		(property "Footprint" "Capacitor_SMD:C_0603_1608Metric"
 			(at 102.5652 149.86 0)
 			(effects

Commit message: v0.2.2
Parts:
- removed Q1: QSZ2TR, symbol Transistor_BJT:Q_Dual_NPN_PNP_B1E2B2C2E1C1
- removed Q2: PMOS, symbol Simulation_SPICE:PMOS
- added Q1: Q_PMOS_GSD, Package_TO_SOT_SMD:SOT-23, symbol Transistor_FET:Q_PMOS_GSD
- added U10: QSZ2TR, Package_TO_SOT_SMD:TSOT-23-5, symbol Transistor_BJT:QSZ2TR
- U6: value Opamp_Dual -> LMR342FVJ; footprint (none) -> Package_SO:TSSOP-8_3x3mm_P0.65mm
Connections:
- net GND: now also U10.5 (CP)
- net VBIAS: now also U10.2 (E)
- net VDD: now also Q1.2 (S)
- net VDDA: now also Q1.3 (D), U10.4 (CN)
- net VDDA_EN: now also Q1.1 (G)
- net at R19.2: now also U10.1 (BP), U10.3 (BN)
Other:
- moved on the sheet: R20
