File: boards/encoder/analog.kicad_sch (KiCad schematic)
At the start: 28 parts, among them Q1 Q_PMOS_GSD, U10 QSZ2TR, U3 CT310, U4 INA826, U5 INA826, U6 LMR342FVJ, U7 AZ431-A

Commit message: Metis-Vela footprint library
Parts:
- U4, U5: footprint Package_SON:SON50P300X300X80-9N200X120 -> metis-vela:SON50P300X300X80-9N200X120
Changed lines of the file:
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@@
 			)
 		)
-		(property "Footprint" "Package_SON:SON50P300X300X80-9N200X120"
+		(property "Footprint" "metis-vela:SON50P300X300X80-9N200X120"
 			(at 109.22 41.91 0)
 			(effects
@@
 			)
 		)
-		(property "Footprint" "Package_SON:SON50P300X300X80-9N200X120"
+		(property "Footprint" "metis-vela:SON50P300X300X80-9N200X120"
 			(at 162.56 41.91 0)
 			(effects

Commit message: v0.2.6
Parts:
- removed R18: 10k, Resistor_SMD:R_0603_1608Metric, symbol Device:R
- removed R22: 50k, Resistor_SMD:R_0603_1608Metric, symbol Device:R
Connections:
- net SIN+: now also U3.1 (SIN-); no longer U3.3 (SIN+)
- net SIN-: now also U3.3 (SIN+); no longer U3.1 (SIN-)
- net VREF+: now also U6.7; no longer U6.1
- net at R17.2, R21.2: now also U6.3 (+); no longer U6.5 (+)
- net at U7.1 (REF): now also R16.2, U6.5 (+), U7.2 (K)
- net at U6.6 (-): now also R24.1; no longer R23.1
- net at R19.1: now also U6.1; no longer U6.7
- net at U6.2 (-): now also R23.1; no longer R24.1

Commit message: v0.2.7
Parts:
- added JP1: SolderJumper_2_Bridged, Jumper:SolderJumper-2_P1.3mm_Bridged_Pad1.0x1.5mm, symbol Jumper:SolderJumper_2_Bridged
Connections:
- net GND: now also JP1.2 (B); no longer C10.2, C11.2, C12.2, C5.2, C6.2, C7.2, C8.1, C9.1, R21.1, U10.5 (CP), U3.4 (GSIN), U3.8 (GCOS), U3.9 (EP), U4.5 (GND), U4.9 (EP), U5.5 (GND), U5.9 (EP), U6.4 (V-), U7.3 (A)
- new net GNDA: C10.2, C11.2, C12.2, C5.2, C6.2, C7.2, C8.1, C9.1, JP1.1 (A), R21.1, U10.5 (CP), U3.4 (GSIN), U3.8 (GCOS), U3.9 (EP), U4.5 (GND), U4.9 (EP), U5.5 (GND), U5.9 (EP), U6.4 (V-), U7.3 (A)
Changed lines of the file:
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@@
 	(wire
 		(pts
-			(xy 224.79 105.41) (xy 217.17 105.41)
-		)
-		(stroke
-			(width 0)
-			(type default)
-		)
-	)
-	(wire
-		(pts
 			(xy 31.75 44.45) (xy 31.75 46.99)
 		)
@@
 	(wire
 		(pts
+			(xy 214.63 105.41) (xy 215.9 105.41)
+		)
+		(stroke
+			(width 0)
+			(type default)
+		)
+	)
+	(wire
+		(pts
 			(xy 106.68 102.87) (xy 106.68 106.68)
 		)
@@
 	(wire
 		(pts
+			(xy 223.52 105.41) (xy 224.79 105.41)
+		)
+		(stroke
+			(width 0)
+			(type default)
+		)
+	)
+	(wire
+		(pts
 			(xy 143.51 41.91) (xy 147.32 41.91)
 		)
@@
 	(wire
 		(pts
-			(xy 217.17 105.41) (xy 217.17 109.22)
+			(xy 214.63 105.41) (xy 214.63 109.22)
 		)
 		(stroke
@@
 	(symbol
 		(lib_id "power:GNDA")
-		(at 217.17 109.22 0)
+		(at 214.63 109.22 0)
 		(unit 1)
 		(exclude_from_sim no)
@@
 		(fields_autoplaced yes)
 		(property "Reference" "#PWR050"
-			(at 217.17 115.57 0)
+			(at 214.63 115.57 0)
 			(effects
 				(font
@@
 		)
 		(property "Value" "GNDA"
-			(at 217.17 114.3 0)
+			(at 214.63 114.3 0)
 			(effects
 				(font
@@
 		)
 		(property "Footprint" ""
-			(at 217.17 109.22 0)
+			(at 214.63 109.22 0)
 			(effects
 				(font
@@
 		)
 		(property "Datasheet" ""
-			(at 217.17 109.22 0)
+			(at 214.63 109.22 0)
 			(effects
 				(font
@@
 		)
 		(property "Description" "Power symbol creates a global label with name \"GNDA\" , analog ground"
-			(at 217.17 109.22 0)
+			(at 214.63 109.22 0)
 			(effects
 				(font
@@
 					(unit 1)
 				)
+			)
+		)
+	)
+	(symbol
+		(lib_id "Jumper:SolderJumper_2_Bridged")
+		(at 219.71 105.41 0)
+		(unit 1)
+		(exclude_from_sim no)
+		(in_bom no)
+		(on_board yes)
+		(dnp no)
+		(fields_autoplaced yes)
+		(property "Reference" "JP1"
+			(at 219.71 99.06 0)
+			(effects
+				(font
+					(size 1.27 1.27)
+				)
+			)
+		)
+		(property "Value" "SolderJumper_2_Bridged"
+			(at 219.71 101.6 0)
+			(effects
+				(font
+					(size 1.27 1.27)
+				)
+			)
+		)
+		(property "Footprint" "Jumper:SolderJumper-2_P1.3mm_Bridged_Pad1.0x1.5mm"
+			(at 219.71 105.41 0)
+			(effects
+				(font
+					(size 1.27 1.27)
+				)
+				(hide yes)
+			)
+		)
+		(property "Datasheet" "~"
+			(at 219.71 105.41 0)
+			(effects
+				(font
+					(size 1.27 1.27)
+				)
+				(hide yes)
+			)
+		)
+		(property "Description" "Solder Jumper, 2-pole, closed/bridged"
+			(at 219.71 105.41 0)
+			(effects
+				(font
+					(size 1.27 1.27)
+				)
+				(hide yes)
+			)
+		)
+		(pin "1"
+		)
+		(pin "2"
+		)
+		(instances
+			(project ""
+				(path "/710faa81-ee23-422b-ba7e-b655a364ab6f/763a463a-636e-4b92-a93e-dd97da54b348"
+					(reference "JP1")
+					(unit 1)
+				)

Commit message: v0.2.9
Parts:
- removed JP1: SolderJumper_2_Bridged, Jumper:SolderJumper-2_P1.3mm_Bridged_Pad1.0x1.5mm, symbol Jumper:SolderJumper_2_Bridged
- renumbered R19 to R18, R20 to R19, R21 to R20, R23 to R21, R24 to R22, U10 to U7, U7 to U8
Connections:
- no-connect marks 0 -> 2
Other:
- note added: "Digital to Analog connections The connection is manual, not via footprint"
- note removed: "Digital to Analog connections"

Commit message: v0.3.10
Parts:
- R14: renamed from R16; value 100 -> 1k
- renumbered R17 to R15, R18 to R16, R19 to R17, R20 to R18, R21 to R19, R22 to R20, R14 to RG1, R15 to RG2
