File: boards/encoder/encoder.kicad_pcb (KiCad board)
At the start: 4 copper layers, 0 parts

Commit message: v0.2.5
Parts:
- added C1: 10u, Capacitor_SMD:C_0603_1608Metric, F.Cu at (141.7, 70.5)
- added C10: 100n, Capacitor_SMD:C_0603_1608Metric, F.Cu at (82.7, 94.5)
- added C11: 100n, Capacitor_SMD:C_0603_1608Metric, F.Cu at (82.7, 97.0)
- added C12: 100n, Capacitor_SMD:C_0603_1608Metric, F.Cu at (164.3, 86.0)
- added C13: 100n, Capacitor_SMD:C_0603_1608Metric, F.Cu at (160.2, 69.2)
- added C14: 100n, Capacitor_SMD:C_0603_1608Metric, F.Cu at (160.2, 71.7)
- added C15: 100n, Capacitor_SMD:C_0603_1608Metric, F.Cu at (160.2, 74.2)
- added C16: 220p, Capacitor_SMD:C_0603_1608Metric, F.Cu at (160.2, 76.7)
- added C17: 220p, Capacitor_SMD:C_0603_1608Metric, F.Cu at (164.3, 69.2)
- added C18: 220p, Capacitor_SMD:C_0603_1608Metric, F.Cu at (164.3, 71.7)
- added C19: 120p, Capacitor_SMD:C_0603_1608Metric, F.Cu at (127.3, 94.4)
- added C2: 100n, Capacitor_SMD:C_0603_1608Metric, F.Cu at (141.7, 73.0)
- added C20: 100u, Capacitor_SMD:C_0603_1608Metric, F.Cu at (127.3, 96.9)
- added C21: 4.7u, Capacitor_SMD:C_0603_1608Metric, F.Cu at (127.3, 99.4)
- added C22: 22u, Capacitor_SMD:C_0603_1608Metric, F.Cu at (127.3, 102.0)
- added C3: 470n, Capacitor_SMD:C_0603_1608Metric, F.Cu at (141.7, 75.5)
- added C4: 20n, Capacitor_SMD:C_0603_1608Metric, F.Cu at (141.7, 78.0)
- added C5: 5600p, Capacitor_SMD:C_0603_1608Metric, F.Cu at (97.5, 66.8)
- added C6: 5600p, Capacitor_SMD:C_0603_1608Metric, F.Cu at (93.2, 80.0)
- added C7: 1u, Capacitor_SMD:C_0603_1608Metric, F.Cu at (93.0, 72.0)
- added C8: 1u, Capacitor_SMD:C_0603_1608Metric, F.Cu at (83.3, 67.7)
- added C9: 1u, Capacitor_SMD:C_0603_1608Metric, F.Cu at (84.8, 83.0)
- added D1: LED, LED_SMD:LED_0603_1608Metric, F.Cu at (153.8, 70.5)
- added D2: LED, LED_SMD:LED_0603_1608Metric, F.Cu at (153.8, 73.1)
- added D3: HT-264USD/UYG-5522, metis-vela:LED_0606_1615Metric, F.Cu at (153.3, 75.1)
- added D4: D_TVS_Dual_AAC, Package_TO_SOT_SMD:SOT-23-3, F.Cu at (172.8, 70.2)
- added D5: D_TVS_Dual_AAC, Package_TO_SOT_SMD:SOT-23-3, F.Cu at (172.8, 74.6)
- added D6: D_TVS_Dual_AAC, Package_TO_SOT_SMD:SOT-23-3, F.Cu at (172.8, 79.1)
- added IC1: TPT480, metis-vela:SON65P300X300X80-9N-D, F.Cu at (180.5, 84.7)
- added J1: SWD, Connector_JST:JST_XH_B4B-XH-A_1x04_P2.50mm_Vertical, F.Cu at (128.7, 62.4)
- added J2: Sensore, Connector_JST:JST_XH_B4B-XH-A_1x04_P2.50mm_Vertical, F.Cu at (128.7, 70.2)
- added J3: Sensore, Connector_JST:JST_XH_B4B-XH-A_1x04_P2.50mm_Vertical, F.Cu at (128.7, 78.0)
- added L1: 1u, Inductor_SMD:L_1210_3225Metric, F.Cu at (132.1, 100.0)
- added Q1: Q_PMOS_GSD, Package_TO_SOT_SMD:SOT-23, F.Cu at (106.2, 64.0)
- added R1: 100k, Resistor_SMD:R_0603_1608Metric, F.Cu at (141.7, 80.5)
- added R10: 4.7k, Resistor_SMD:R_0603_1608Metric, F.Cu at (149.7, 73.0)
- added R11: 4.7k, Resistor_SMD:R_0603_1608Metric, F.Cu at (149.7, 75.5)
- added R12: 470, Resistor_SMD:R_0603_1608Metric, F.Cu at (94.0, 66.8)
- added R13: 470, Resistor_SMD:R_0603_1608Metric, F.Cu at (90.0, 80.0)
- added R14: 98.8k, Resistor_SMD:R_0603_1608Metric, F.Cu at (86.0, 67.7)
- added R15: 98.8k, Resistor_SMD:R_0603_1608Metric, F.Cu at (88.2, 75.5)
- added R16: 100, Resistor_SMD:R_0603_1608Metric, F.Cu at (81.1, 64.5)
- added R17: 10k, Resistor_SMD:R_0603_1608Metric, F.Cu at (74.8, 75.3)
- added R18: 10k, Resistor_SMD:R_0603_1608Metric, F.Cu at (80.2, 67.7)
- added R19: 100, Resistor_SMD:R_0603_1608Metric, F.Cu at (77.7, 79.8)
- added R2: 47k, Resistor_SMD:R_0603_1608Metric, F.Cu at (141.7, 83.0)
- added R20: 10k, Resistor_SMD:R_0603_1608Metric, F.Cu at (111.3, 64.0)
- added R21: 10k, Resistor_SMD:R_0603_1608Metric, F.Cu at (74.8, 71.7)
- added R22: 50k, Resistor_SMD:R_0603_1608Metric, F.Cu at (78.0, 71.8)
- added R23: 100, Resistor_SMD:R_0603_1608Metric, F.Cu at (81.7, 79.8)
- added R24: 100, Resistor_SMD:R_0603_1608Metric, F.Cu at (86.2, 73.0)
- added R25: 60, Resistor_SMD:R_0603_1608Metric, F.Cu at (164.3, 74.2)
- added R26: 60, Resistor_SMD:R_0603_1608Metric, F.Cu at (164.3, 76.7)
- added R27: 60, Resistor_SMD:R_0603_1608Metric, F.Cu at (168.3, 69.2)
- added R28: 60, Resistor_SMD:R_0603_1608Metric, F.Cu at (168.3, 71.7)
- added R29: 60, Resistor_SMD:R_0603_1608Metric, F.Cu at (168.3, 74.2)
- added R3: 47k, Resistor_SMD:R_0603_1608Metric, F.Cu at (145.7, 70.5)
- added R30: 60, Resistor_SMD:R_0603_1608Metric, F.Cu at (168.3, 76.7)
- added R31: 455k, Resistor_SMD:R_0603_1608Metric, F.Cu at (127.3, 104.5)
- added R32: 95k, Resistor_SMD:R_0603_1608Metric, F.Cu at (127.3, 107.0)
- added R4: 499k, Resistor_SMD:R_0603_1608Metric, F.Cu at (145.7, 73.0)
- added R5: 65, Resistor_SMD:R_0603_1608Metric, F.Cu at (145.7, 75.5)
- added R6: 65, Resistor_SMD:R_0603_1608Metric, F.Cu at (145.7, 78.0)
- added R7: 150, Resistor_SMD:R_0603_1608Metric, F.Cu at (145.7, 80.5)
- added R8: 65, Resistor_SMD:R_0603_1608Metric, F.Cu at (145.7, 83.0)
- added R9: 4.7k, Resistor_SMD:R_0603_1608Metric, F.Cu at (149.7, 70.5)
- added RV1: 10k, Potentiometer_SMD:Potentiometer_Bourns_TC33X_Vertical, F.Cu at (133.5, 94.0)
- added SW1: SW_SPST, metis-vela:SW_DS04-254-1-01BK-SMT, F.Cu at (146.2, 61.6)
- added SW2: SW_SPST, metis-vela:SW_DS04-254-1-01BK-SMT, F.Cu at (146.2, 66.7)
- added SW3: SW_Push, metis-vela:SW_TS04-66-65-BK-260-SMT, F.Cu at (132.2, 86.2)
- added SW4: 204_211ST, metis-vela:SW4_204-211ST_CTS, F.Cu at (164.5, 63.5)
- added U1: MSPM0G310x, metis-vela:RHB0032D-IPC_A, F.Cu at (107.5, 72.5)
- added U10: QSZ2TR, Package_TO_SOT_SMD:TSOT-23-5, F.Cu at (95.5, 75.6)
- added U2: M24C08, metis-vela:SO8N_4X5X1P27_STM, F.Cu at (144.0, 87.6)
- added U3: CT310, Package_DFN_QFN:DFN-8-1EP_2x2mm_P0.5mm_EP0.8x1.6mm, F.Cu at (90.0, 73.0)
- added U4: INA826, metis-vela:SON50P300X300X80-9N200X120, F.Cu at (90.0, 68.0)
- added U5: INA826, metis-vela:SON50P300X300X80-9N200X120, F.Cu at (86.8, 78.8)
- added U6: LMR342FVJ, Package_SO:TSSOP-8_3x3mm_P0.65mm, F.Cu at (82.2, 73.2)
- added U7: AZ431-A, Package_TO_SOT_SMD:SOT-23-3, F.Cu at (75.9, 67.5)
- added U8: TCAN1044V, metis-vela:SOT-23-THIN-8_DDF_TEX, F.Cu at (160.9, 80.3)
- added U9: TPS62A02A, Package_TO_SOT_SMD:SOT-563, F.Cu at (131.0, 103.8)
Routing:
- net GND: track 0.00 -> 38.6 mm, vias 0 -> 5
- net /VBIAS: track 0.00 -> 34.3 mm
- net /VREF+: track 0.00 -> 25.9 mm, vias 0 -> 3
- net Net-(U10-BN): track 0.00 -> 22.7 mm, vias 0 -> 3
- net /Analog/SIN-: track 0.00 -> 15.7 mm
- net /Analog/COS-: track 0.00 -> 12.7 mm
- net Net-(U6A-+): track 0.00 -> 11.5 mm
- net Net-(U6B--): track 0.00 -> 8.97 mm
- net Net-(U6B-+): track 0.00 -> 8.93 mm
- net Net-(R19-Pad1): track 0.00 -> 7.97 mm
- net /Analog/COS+: track 0.00 -> 7.84 mm
- net /Analog/SIN+: track 0.00 -> 6.58 mm, vias 0 -> 2
- net Net-(U7-REF): track 0.00 -> 6.42 mm
- net Net-(U6A--): track 0.00 -> 4.46 mm
- net /COS_IN: track 0.00 -> 3.95 mm
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Other:
- board text added: "${REFERENCE}"

Commit message: v0.2.6
Parts:
- removed R18: 10k, Resistor_SMD:R_0603_1608Metric
- removed R22: 50k, Resistor_SMD:R_0603_1608Metric
- added H1: MountingHole, MountingHole:MountingHole_3.2mm_M3_DIN965_Pad, F.Cu at (18.2, 17.2)
- added H2: MountingHole, MountingHole:MountingHole_3.2mm_M3_DIN965_Pad, F.Cu at (18.2, 24.3)
- added H3: MountingHole, MountingHole:MountingHole_3.2mm_M3_DIN965_Pad, F.Cu at (18.2, 31.5)
- added H4: MountingHole, MountingHole:MountingHole_3.2mm_M3_DIN965_Pad, F.Cu at (28.6, 62.5)
- moved D1 139.7 mm to (16.7, 43.5)
- moved D2 139.7 mm to (16.7, 46.1)
- moved D3 136.9 mm to (20.2, 43.0)
- moved IC1 131.6 mm to (58.6, 35.0)
- moved R3 117.5 mm to (42.3, 14.9)
- moved R4 117.5 mm to (42.3, 17.4)
- moved R5 117.5 mm to (42.3, 19.9)
- moved R6 117.5 mm to (42.3, 22.4)
- moved R7 117.5 mm to (42.3, 24.9)
- moved R8 117.5 mm to (42.3, 27.4)
- moved R10 117.5 mm to (46.3, 17.4)
- moved R11 117.5 mm to (46.3, 19.9)
- moved R9 117.5 mm to (46.3, 14.9)
- moved C1 117.5 mm to (38.2, 14.9)
- moved C2 117.5 mm to (38.2, 17.4)
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Connections:
- R16 pad 2: Net-(U6A-+) -> Net-(U6B-+)
- R17 pad 2: Net-(U6B-+) -> Net-(U6A-+)
- R21 pad 2: Net-(U6B-+) -> Net-(U6A-+)
- R23 pad 1: Net-(U6B--) -> Net-(U6A--)
- R24 pad 1: Net-(U6A--) -> Net-(U6B--)
- U1 pad 26: unconnected-(U1-PA22_A0_7-Pad26) -> /COS_IN
- U1 pad 28: /COS_IN -> /VDDA_EN
- U1 pad 9: /VDDA_EN -> unconnected-(U1-PA5_HFXIN_FCC_IN-Pad9)
- U3 pad 1: /Analog/SIN- -> /Analog/SIN+
- U3 pad 3: /Analog/SIN+ -> /Analog/SIN-
- U6 pad 1: /VREF+ -> Net-(R19-Pad1)
- U6 pad 7: Net-(R19-Pad1) -> /VREF+
- U7 pad 1: Net-(U7-REF) -> Net-(U6B-+)
- U7 pad 2: Net-(U6A-+) -> Net-(U6B-+)
Routing:
- net /VBIAS: track 34.3 -> 7.88 mm, vias 0 -> 4
- net Net-(U10-BN): track 22.7 -> 0.00 mm, vias 3 -> 0
- net VDDA: track 0.00 -> 15.2 mm, vias 0 -> 2
- net /VREF+: track 25.9 -> 12.1 mm, vias 3 -> 4
- net Net-(U6A-+): track 11.5 -> 0.00 mm
- net /Analog/COS-: track 12.7 -> 3.13 mm
- net Net-(U6B--): track 8.97 -> 0.00 mm
- net Net-(U6B-+): track 8.93 -> 0.00 mm
- net Net-(R19-Pad1): track 7.97 -> 0.00 mm
- net /Analog/SIN-: track 15.7 -> 7.99 mm
- net Net-(U7-REF): track 6.42 -> 0.00 mm
- net Net-(U6A--): track 4.46 -> 0.00 mm
- net /COS_IN: track 3.95 -> 8.03 mm
- net /BOOT: track 0.00 -> 3.86 mm, vias 0 -> 1
- net /Analog/SIN+: track 6.58 -> 3.10 mm, vias 2 -> 0
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- added copper zone on F.Cu, net /VBIAS
- added copper zone on In1.Cu, net /VBIAS
Other:
- board text removed: "${REFERENCE}"

Commit message: v0.2.7
Parts:
- added JP1: SolderJumper_2_Bridged, Jumper:SolderJumper-2_P1.3mm_Bridged_Pad1.0x1.5mm, F.Cu at (64.8, 41.1)
- C19, C20, C21, C22, D3, J1, J2, J3, L1, R2, R3, R31, R32, R5, R6, RV1, SW1, SW2, U9: moved to B.Cu
- moved C1 140.4 mm to (170.9, 61.0)
- moved C2 140.3 mm to (170.9, 63.0)
- moved H4 136.1 mm to (163.4, 81.5)
- moved J2 132.5 mm to (155.3, 50.0)
- moved D3 121.7 mm to (125.7, 103.6)
- moved J1 121.2 mm to (141.9, 50.0)
- moved R5 118.3 mm to (124.7, 104.7), turned to 90 degrees
- moved H2 118.0 mm to (121.4, 81.5)
- moved R6 117.9 mm to (126.7, 104.7), turned to 90 degrees
- moved H1 108.1 mm to (121.4, 49.5)
- moved J3 104.7 mm to (128.5, 50.0)
- moved IC1 94.0 mm to (150.0, 57.2)
- moved R2 93.7 mm to (82.7, 109.9), turned to -90 degrees
- moved SW1 83.3 mm to (79.5, 106.0), turned to 90 degrees
- moved C19 79.2 mm to (90.9, 109.9), turned to 90 degrees
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Connections:
- C10 pad 2: GND -> GNDA
- C11 pad 2: GND -> GNDA
- C12 pad 2: GND -> GNDA
- C5 pad 2: GND -> GNDA
- C6 pad 2: GND -> GNDA
- C7 pad 2: GND -> GNDA
- C8 pad 1: GND -> GNDA
- C9 pad 1: GND -> GNDA
- D4 pad 1: /Transmission Lines/RS485_A -> /Transmission Lines/RS485_1-
- D4 pad 2: /Transmission Lines/RS485_B -> /Transmission Lines/RS485_1+
- D5 pad 1: /Transmission Lines/RS485_Z -> /Transmission Lines/RS485_2-
- D5 pad 2: /Transmission Lines/RS485_Y -> /Transmission Lines/RS485_2+
- IC1 pad 5: /Transmission Lines/RS485_Y -> /Transmission Lines/RS485_2-
- IC1 pad 6: /Transmission Lines/RS485_Z -> /Transmission Lines/RS485_2+
- IC1 pad 7: /Transmission Lines/RS485_B -> /Transmission Lines/RS485_1-
- IC1 pad 8: /Transmission Lines/RS485_A -> /Transmission Lines/RS485_1+
- R21 pad 1: GND -> GNDA
- R25 pad 1: /Transmission Lines/RS485_A -> /Transmission Lines/RS485_1+
- R26 pad 1: /Transmission Lines/RS485_Z -> /Transmission Lines/RS485_2+
- R29 pad 2: /Transmission Lines/RS485_B -> /Transmission Lines/RS485_1-
- R30 pad 2: /Transmission Lines/RS485_Y -> /Transmission Lines/RS485_2-
- U1 pad 10: /CAN_STB -> unconnected-(U1-PA6_HFCLK_IN_HFXOUT-Pad10)
- U1 pad 19: /SIN_IN -> /VDDA_EN
- U1 pad 20: /VBIAS -> /SIN_IN
- U1 pad 21: unconnected-(U1-PA17_A1_2-Pad21) -> /VBIAS
- U1 pad 25: GND -> GNDA
- U1 pad 28: /VDDA_EN -> unconnected-(U1-PA24_A0_3-Pad28)
- U1 pad 29: unconnected-(U1-PA25_A0_2-Pad29) -> /CAN_STB
- U1 pad 9: unconnected-(U1-PA5_HFXIN_FCC_IN-Pad9) -> /ROM_WC
- U10 pad 5: GND -> GNDA
- U3 pad 4: GND -> GNDA
- U3 pad 8: GND -> GNDA
- U3 pad 9: GND -> GNDA
- U4 pad 5: GND -> GNDA
- U4 pad 9: GND -> GNDA
- U5 pad 5: GND -> GNDA
- U5 pad 9: GND -> GNDA
- U6 pad 4: GND -> GNDA
- U7 pad 3: GND -> GNDA
Routing:
- net /VREF+: track 12.1 -> 52.4 mm
- net GND: track 38.8 -> 6.94 mm, vias 1 -> 2
- net /UART_RX: track 0.00 -> 31.7 mm
- net /UART_TX: track 0.00 -> 28.4 mm
- net GNDA: track 0.00 -> 25.2 mm, vias 0 -> 13
- net Net-(U6A-+): track 0.00 -> 17.4 mm
- net /AY_TX: track 0.00 -> 13.2 mm
- net /VBIAS: track 7.88 -> 19.7 mm
- net Net-(U6B-+): track 0.00 -> 11.0 mm
- net /AY_RX: track 0.00 -> 9.75 mm
- net /Transmission Lines/RS485_1+: track 0.00 -> 8.78 mm
- net /Transmission Lines/RS485_1-: track 0.00 -> 8.77 mm
- net /Transmission Lines/RS485_2-: track 0.00 -> 8.77 mm
- net /Transmission Lines/RS485_2+: track 0.00 -> 8.76 mm
- net Net-(R19-Pad1): track 0.00 -> 8.23 mm
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- added copper zone on In1.Cu, net GNDA
Other:
- board outline added: 50 x 40 mm
- board text added: "${REFERENCE}"

Commit message: v0.2.8
Parts:
- added J5: RS485, Connector_JST:JST_XH_B4B-XH-A_1x04_P2.50mm_Vertical, B.Cu at (163.5, 48.5)
- R10, R11, R9, U2: moved to B.Cu
- moved C3 115.1 mm to (144.2, 65.0), turned to -90 degrees
- moved R1 45.9 mm to (146.3, 57.4)
- moved R25 42.0 mm to (150.7, 49.4), turned to 0 degrees
- moved D4 42.0 mm to (158.4, 50.3)
- moved C16 42.0 mm to (154.2, 50.3)
- moved R29 40.8 mm to (150.7, 51.3), turned to 180 degrees
- moved D5 40.0 mm to (158.4, 54.4)
- moved C17 40.0 mm to (154.2, 54.4)
- moved R26 39.9 mm to (150.7, 53.3), turned to 0 degrees
- moved R30 39.0 mm to (150.7, 55.5), turned to 180 degrees
- moved J2 28.0 mm to (146.8, 23.3)
- moved C2 25.5 mm to (145.5, 60.5), turned to 90 degrees
- moved C1 23.3 mm to (147.6, 60.5), turned to 90 degrees
- moved J1 20.5 mm to (146.8, 30.1)
- moved R11 6.23 mm to (65.8, 73.8)
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Routing:
- net VDDA: track 8.76 -> 43.7 mm
- net /UART_RX: track 31.7 -> 0.00 mm
- net /UART_TX: track 28.4 -> 0.00 mm
- net /Transmission Lines/RS485_2-: track 8.77 -> 17.6 mm
- net /Transmission Lines/RS485_1+: track 8.78 -> 17.3 mm
- net /Transmission Lines/RS485_2+: track 8.76 -> 17.0 mm
- net /Transmission Lines/RS485_1-: track 8.77 -> 16.9 mm
- net GND: track 6.94 -> 13.5 mm, vias 2 -> 6
- net +3.3V: track 0.00 -> 4.97 mm, vias 0 -> 1
- net /ROSC: track 0.00 -> 3.59 mm
- net /RS485_RX: track 4.79 -> 8.33 mm
- net /LED1_OUT: track 0.00 -> 3.46 mm, vias 0 -> 1
- net /RS485_TX: track 4.09 -> 7.52 mm
- net /LED2_OUT: track 0.00 -> 3.14 mm, vias 0 -> 1
- net /RESET: track 0.00 -> 3.01 mm, vias 0 -> 1
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- added copper zone on In1.Cu, net GND
- added copper zone on In2.Cu, net GND

Commit message: v0.2.9
Parts:
- removed the H3 at (18.2, 31.5)
- removed JP1: SolderJumper_2_Bridged, Jumper:SolderJumper-2_P1.3mm_Bridged_Pad1.0x1.5mm
- removed the R27 at (73.3, 25.1)
- removed the R28 at (73.3, 22.5)
- removed R31: 455k, Resistor_SMD:R_0603_1608Metric
- removed R32: 95k, Resistor_SMD:R_0603_1608Metric
- removed the U8 at (94.5, 72.5)
- added J4: CANbus, Connector_JST:JST_XH_B2B-XH-A_1x02_P2.50mm_Vertical, B.Cu at (162.9, 62.2)
- added J6: PWR, Connector_JST:JST_XH_B2B-XH-A_1x02_P2.50mm_Vertical, B.Cu at (162.9, 70.9)
- added R25: 60, Resistor_SMD:R_0603_1608Metric, B.Cu at (158.0, 66.4)
- added R26: 60, Resistor_SMD:R_0603_1608Metric, B.Cu at (158.0, 60.5)
- added R29: 455k, Resistor_SMD:R_0603_1608Metric, B.Cu at (95.0, 23.8)
- added R30: 95k, Resistor_SMD:R_0603_1608Metric, B.Cu at (95.0, 21.3)
- added U10: TPS62A02A, Package_TO_SOT_SMD:SOT-563, B.Cu at (98.8, 24.5)
- C14, C15, C18, C4, D1, D2, D6, R4, R7, R8, SW3, SW4: moved to B.Cu
- U9: value TPS62A02A -> TCAN1044V; footprint Package_TO_SOT_SMD:SOT-563 -> metis-vela:SOT-23-THIN-8_DDF_TEX
- moved D1 143.7 mm to (157.8, 70.5), turned to 90 degrees
- moved R7 125.5 mm to (157.8, 74.0), turned to -90 degrees
- moved C14 105.8 mm to (152.8, 60.4), turned to 180 degrees
- moved C15 102.7 mm to (149.4, 63.5), turned to -90 degrees
- moved D2 102.6 mm to (117.8, 28.7)
- moved R4 97.3 mm to (134.2, 59.9), turned to 90 degrees
- moved SW3 97.0 mm to (127.0, 58.1)
- moved C4 96.3 mm to (134.2, 56.5), turned to 90 degrees
- moved C13 96.3 mm to (145.4, 49.6)
- moved U2 94.9 mm to (138.9, 28.7), turned to 180 degrees
- moved C20 88.2 mm to (95.0, 31.3), turned to 0 degrees
- moved L1 86.2 mm to (99.8, 28.2)
- moved C22 83.8 mm to (95.0, 26.3), turned to 0 degrees
- moved R9 83.6 mm to (132.5, 28.8), turned to 180 degrees
- moved C18 83.1 mm to (146.9, 54.3), turned to 90 degrees
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- renumbered H4 to H3, R19 to R18, R20 to R19, R21 to R20, R23 to R21, R24 to R22, R25 to R23, R26 to R24, R29 to R27, R30 to R28, U10 to U7, U7 to U8
Connections:
- C18 pad 2: Net-(C18-Pad2) -> Net-(SW4-2)
- D6 pad 1: /Transmission Lines/CAN_H -> /Transmission Lines/CAN_L
- D6 pad 2: /Transmission Lines/CAN_L -> /Transmission Lines/CAN_H
- H1 pad 1: (no net) -> GND
- H2 pad 1: (no net) -> GND
- H3 pad 1: (no net) -> GND
- J1 pad 2: /SWDIO -> /SWCLK
- J1 pad 3: /SWCLK -> /SWDIO
- SW4 pad 1: /Transmission Lines/CAN_H -> Net-(SW4-3)
- SW4 pad 2: /Transmission Lines/CAN_L -> Net-(SW4-1)
- SW4 pad 4: Net-(R27-Pad2) -> Net-(SW4-2)
- U1 pad 1: /LED1_OUT -> /LED2_OUT
- U1 pad 2: /LED2_OUT -> /LED1_OUT
- U9 pad 1: GND -> /CAN_TX
- U9 pad 2: /PSU/PWR_SW -> GND
- U9 pad 4: /PWR_EN -> /CAN_RX
- U9 pad 5: /PSU/PWR_FB -> +3.3V
- U9 pad 6: /RESET -> /Transmission Lines/CAN_L
Routing:
- net VDD: track 0.00 -> 91.4 mm, vias 0 -> 1
- net /UART_RX: track 0.00 -> 31.4 mm, vias 0 -> 2
- net /UART_TX: track 0.00 -> 28.1 mm, vias 0 -> 2
- net /SWDIO: track 3.37 -> 23.4 mm
- net /SWCLK: track 2.19 -> 21.5 mm
- net /RESET: track 3.01 -> 21.3 mm, vias 1 -> 2
- net /CAN_STB: track 0.00 -> 17.9 mm, vias 0 -> 1
- net Net-(SW4-3): track 0.00 -> 15.1 mm, vias 0 -> 2
- net /VDDA_EN: track 0.00 -> 14.2 mm
- net /CAN_TX: track 0.00 -> 14.0 mm, vias 0 -> 1
- net /CAN_RX: track 0.00 -> 14.0 mm, vias 0 -> 1
- net GND: track 13.5 -> 26.5 mm, vias 6 -> 13
- net /Transmission Lines/CAN_L: track 0.00 -> 11.2 mm
- net /Transmission Lines/CAN_H: track 0.00 -> 11.2 mm
- net /PWR_EN: track 8.00 -> 0.00 mm
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Other:
- board text removed: "${REFERENCE}"

Commit message: v0.2.10
Parts:
- U2: footprint metis-vela:SO8N_4X5X1P27_STM -> metis-vela:UFDFPN5_1P7X1P4_STM
- moved R2 46.6 mm to (134.2, 68.6), turned to -90 degrees
- moved SW1 41.4 mm to (127.2, 68.6), turned to 180 degrees
- moved R8 40.9 mm to (148.1, 59.6)
- moved D2 40.7 mm to (146.5, 57.6), turned to 180 degrees
- moved R30 38.0 mm to (74.1, 53.0), turned to 90 degrees
- moved R29 34.5 mm to (76.6, 53.0), turned to 90 degrees
- moved U10 32.8 mm to (77.2, 49.2), turned to 90 degrees
- moved C22 31.1 mm to (79.1, 53.0), turned to 90 degrees
- moved C21 27.6 mm to (81.6, 53.0), turned to 90 degrees
- moved L1 27.4 mm to (81.0, 48.2), turned to 90 degrees
- moved C20 24.2 mm to (84.1, 53.0), turned to 90 degrees
- moved U2 22.4 mm to (142.2, 50.8), turned to -90 degrees
- moved R11 22.2 mm to (140.2, 47.6), turned to 90 degrees
- moved R9 22.1 mm to (144.2, 47.6), turned to 90 degrees
- moved RV1 21.1 mm to (85.5, 47.8), turned to 90 degrees
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Connections:
- U2 pad 1: unconnected-(U2-NC-Pad1) -> +3.3V
- U2 pad 2: unconnected-(U2-NC-Pad2) -> GND
- U2 pad 3: GND -> /I2C_SDA
- U2 pad 4: GND -> /I2C_SCL
- U2 pad 5: /I2C_SDA -> /ROM_WC
Routing:
- net +3.3V: track 12.7 -> 27.2 mm
- net GND: track 26.5 -> 34.8 mm, vias 13 -> 19
- net /I2C_SDA: track 5.82 -> 13.9 mm, vias 1 -> 3
- net VDD: track 91.4 -> 99.0 mm
- net /I2C_SCL: track 4.68 -> 11.3 mm
- net /ROM_WC: track 4.35 -> 10.6 mm
- net /RESET: track 21.3 -> 26.3 mm, vias 2 -> 1
- net /PWR_EN: track 0.00 -> 2.92 mm
- net Net-(D2-K): track 0.00 -> 2.00 mm
