File: boards/encoder/encoder.kicad_pcb (KiCad board)
At the start: 4 copper layers, 50 x 40 mm, 85 parts, among them IC1 TPT480, J1 SWD, J2 Sensore, J3 Sensore, J4 CANbus, J5 RS485, J6 PWR, Q1 Q_PMOS_GSD, SW1 SW_SPST, SW2 SW_SPST, SW3 SW_Push, SW4 204_211ST, U1 MSPM0G310x, U10 TPS62A02A, U2 M24C08, U3 CT310, U4 INA826, U5 INA826, U6 LMR342FVJ, U7 QSZ2TR, U8 AZ431-A, U9 TCAN1044V

Commit message: v0.3.0
Parts:
- C20: footprint Capacitor_SMD:C_0603_1608Metric -> Capacitor_SMD:C_1206_3216Metric; moved to F.Cu
- U1: footprint metis-vela:RHB0032D-IPC_A -> Package_DFN_QFN:Texas_RHB0032E_VQFN-32-1EP_5x5mm_P0.5mm_EP3.45x3.45mm_ThermalVias
- moved C20 78.4 mm to (160.1, 72.2)
- moved U10 75.3 mm to (149.4, 70.6), turned to 180 degrees
- moved L1 75.1 mm to (152.7, 70.6)
- moved C22 71.7 mm to (149.1, 68.3), turned to 180 degrees
- moved C21 70.4 mm to (149.1, 72.9), turned to 180 degrees
- moved R30 69.8 mm to (142.0, 69.0)
- moved R29 69.3 mm to (144.0, 69.0), turned to -90 degrees
- moved RV1 63.7 mm to (144.1, 72.9), turned to 0 degrees
- moved C19 61.5 mm to (146.0, 69.0), turned to -90 degrees
- moved D1 3.50 mm to (157.8, 74.0), turned to -90 degrees
- moved R7 3.50 mm to (157.8, 70.5), turned to 90 degrees
- moved R5 0.50 mm to (143.2, 60.3)
- moved R6 0.50 mm to (145.2, 60.3)
Connections:
- J6 pad 1: VDD -> GND
- J6 pad 2: GND -> VDD
Routing:
- net +3.3V: track 27.2 -> 103.8 mm, vias 2 -> 8
- net VDD: track 99.0 -> 126.5 mm
- net /PWR_EN: track 2.92 -> 19.1 mm, vias 0 -> 2
- net GND: track 34.8 -> 48.6 mm, vias 19 -> 24
- net Net-(C19-Pad2): track 0.00 -> 6.80 mm
- net /RESET: track 26.3 -> 32.8 mm
- net /PSU/PWR_FB: track 0.00 -> 5.69 mm
- net /UART_RX: track 31.4 -> 27.8 mm
- net /PSU/PWR_SW: track 0.00 -> 3.15 mm
- net Net-(R30-Pad1): track 0.00 -> 2.20 mm
- net Net-(U6B-+): track 11.0 -> 12.9 mm
- net /UART_TX: track 28.1 -> 29.1 mm
- net GNDA: track 25.2 -> 25.7 mm

Commit message: v0.3.1
Other:
- board text added: "WANDA BTM"
- board text added: "WANDA TOP"
Changed lines of the file:
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@@
 		(tags "resistor")
 		(property "Reference" "R23"
-			(at 3.051 -0.426 0)
+			(at -0.125 -1.475 0)
 			(layer "F.SilkS")
 			(effects
@@
 		(tags "resistor")
 		(property "Reference" "R16"
-			(at 2.3 -1.2625 180)
+			(at 2.35 0.0375 180)
 			(layer "F.SilkS")
 			(effects
@@
 		(tags "capacitor")
 		(property "Reference" "C10"
-			(at 0.617101 1.407899 0)
+			(at 0.117101 1.407899 0)
 			(layer "F.SilkS")
 			(effects
@@
 		(tags "capacitor")
 		(property "Reference" "C5"
-			(at -0.607899 1.407899 0)
+			(at -0.007899 1.407899 0)
 			(layer "F.SilkS")
 			(effects
@@
 		(tags "resistor")
 		(property "Reference" "R14"
-			(at -2.207899 -0.360399 180)
+			(at -2.207899 -0.060399 180)
 			(layer "F.SilkS")
 			(effects
@@
 		(tags "resistor")
 		(property "Reference" "R19"
-			(at -2.5 0.6 180)
+			(at -2.5 -0.0375 180)
 			(layer "F.SilkS")
 			(effects
@@
 		(tags "capacitor")
 		(property "Reference" "C3"
-			(at 0 -1.43 180)
+			(at 0.025 -1.7 180)
 			(layer "F.SilkS")
 			(effects
@@
 		(tags "capacitor")
 		(property "Reference" "C12"
-			(at 2.25 -0.4625 180)
+			(at -2.25 -0.0625 180)
 			(layer "F.SilkS")
 			(effects
@@
 		(tags "resistor")
 		(property "Reference" "R21"
-			(at -1.2 -1.6 0)
+			(at -1 -1.5 0)
 			(layer "F.SilkS")
 			(effects
@@
 		(tags "capacitor")
 		(property "Reference" "C16"
-			(at -1.726 -1.424 0)
+			(at -0.05 1.225 0)
 			(layer "F.SilkS")
 			(effects
@@
 		(tags "capacitor")
 		(property "Reference" "C9"
-			(at -2.5 0.7 0)
+			(at 0 -1.3 0)
 			(layer "F.SilkS")
 			(effects
@@
 		(tags "capacitor")
 		(property "Reference" "C6"
-			(at 0.7 1.782899 0)
+			(at 0 1.682899 0)
 			(layer "F.SilkS")
 			(effects
@@
 		(tags "capacitor")
 		(property "Reference" "C17"
-			(at -1.726 -1.474 0)
+			(at -0.05 -1.325 0)
 			(layer "F.SilkS")
 			(effects
@@
 		(tags "capacitor")
 		(property "Reference" "C7"
-			(at 2.300001 -0.1 180)
+			(at -0.099999 -1.5 0)
 			(layer "F.SilkS")
 			(effects
@@
 		(tags "resistor")
 		(property "Reference" "R15"
-			(at 0.017101 2.342101 180)
+			(at -0.082899 2.142101 180)
 			(layer "F.SilkS")
 			(effects
@@
 		(tags "capacitor")
 		(property "Reference" "C1"
-			(at 1.85 0 0)
+			(at 1.95 0 0)
 			(layer "F.SilkS")
 			(effects
@@
 		(tags "resistor")
 		(property "Reference" "R28"
-			(at -2.551 -0.324 0)
+			(at -1.575 -1.275 0)
 			(layer "F.SilkS")
 			(effects
@@
 		(tags "Texas VQFN NoLead")
 		(property "Reference" "U1"
-			(at 0 -3.83 180)
+			(at -0.051247 3.950001 180)
 			(layer "F.SilkS")
 			(effects
@@
 		(tags "204-211ST ")
 		(property "Reference" "SW4"
-			(at 0 0 0)
+			(at 0 4.7 0)
 			(unlocked yes)
 			(layer "B.SilkS")
@@
 		)
 		(fp_text user "${REFERENCE}"
-			(at 0 0 0)
+			(at 0 4.7 0)
 			(unlocked yes)
 			(layer "B.Fab")
@@
 		(at 127.15 68.6 180)
 		(property "Reference" "SW1"
-			(at 0.175 2.885 0)
+			(at 7.55 0.1 90)
 			(layer "B.SilkS")
 			(effects
@@
 		(at 127.05 58.15)
 		(property "Reference" "SW3"
-			(at -0.05 -4.15 180)
+			(at -7.55 0.05 270)
 			(layer "B.SilkS")
 			(effects
@@
 		(at 127.15 64 180)
 		(property "Reference" "SW2"
-			(at 0.0625 -2.9 0)
+			(at 7.65 0 90)
 			(layer "B.SilkS")
 			(effects
@@
 		(tags "TCAN1044VDDFR ")
 		(property "Reference" "U9"
-			(at 0 0 180)
+			(at 0 2.65 0)
 			(unlocked yes)
 			(layer "B.SilkS")
@@
 		)
 		(fp_text user "${REFERENCE}"
-			(at 0 0 180)
+			(at 0 2.65 180)
 			(unlocked yes)
 			(layer "B.Fab")
@@
 		(tags "SOT TO_SOT_SMD")
 		(property "Reference" "D6"
-			(at 0 2.4 0)
+			(at 1.8375 2.05 0)
 			(layer "B.SilkS")
 			(effects
@@
 		(tags "capacitor")
 		(property "Reference" "C18"
-			(at -0.055 1.5 90)
+			(at -0.055 1.2 90)
 			(layer "B.SilkS")
 			(effects
@@
 		(layer "F.Fab")
 	)
+	(gr_text "WANDA TOP\n"
+		(at 151.5 83.3 0)
+		(layer "F.SilkS")
+		(effects
+			(font
+				(size 1 1)
+				(thickness 0.25)
+				(bold yes)
+			)
+			(justify left bottom)
+		)
+	)
+	(gr_text "WANDA BTM\n"
+		(at 161 84.8 0)
+		(layer "F.SilkS")
+		(effects
+			(font
+				(size 1 1)
+				(thickness 0.25)
+				(bold yes)
+			)
+			(justify left bottom mirror)
+		)
+	)
 	(dimension
 		(type orthogonal)
@@
 		(start 134.175 69.425)
 		(end 125.1 78.5)
-		(width 0.2)
+		(width 0.4)
 		(layer "B.Cu")
 		(net 10)
@@
 		(net 31)
 	)
+	(via
+		(at 139.3 56.8)
+		(size 0.6)
+		(drill 0.3)
+		(layers "F.Cu" "B.Cu")
+		(net 31)
+	)
 	(segment
 		(start 139.4 65.7)
@@
 		(net 31)
 	)
-	(via blind
-		(at 139.3 56.8)
-		(size 0.6)
-		(drill 0.3)
-		(layers "In2.Cu" "B.Cu")
-		(net 31)
-	)

Commit message: v.0.3.3
Parts:
- moved R10 2.55 mm to (142.2, 50.2)
- moved R11 2.55 mm to (140.2, 50.2)
- moved R9 2.55 mm to (144.2, 50.2)
- moved U2 2.55 mm to (142.2, 53.4)
- moved R1 0.20 mm to (146.3, 57.2)
Routing:
- net +3.3V: track 103.8 -> 100.7 mm
- net /I2C_SDA: track 13.6 -> 11.1 mm
- net /I2C_SCL: track 11.3 -> 8.75 mm
- net /ROM_WC: track 10.6 -> 8.08 mm
Other:
- board text added: "WANDA r1.0"
- board text added: "WayWayWay"
- board text removed: "WANDA BTM"
- board text removed: "WANDA TOP"

Commit message: v0.3.4
Parts:
- renumbered D2 to 3v3, SW2 to BOOT, SW1 to PWR, D1 to PWR, SW3 to RESET
Changed lines of the file:
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@@
 			(unlocked yes)
 			(layer "B.SilkS")
+			(hide yes)
 			(effects
 				(font
@@
 			)
 		)
-		(fp_text user "*"
-			(at -4.7625 2.0828 0)
-			(layer "B.Fab")
+		(fp_text user "CAN TERM"
+			(at 0 4.7 0)
+			(unlocked yes)
+			(layer "B.SilkS")
 			(effects
 				(font
@@
 			)
 		)
-		(fp_text user "ON"
-			(at 5.0165 5.1562 0)
-			(unlocked yes)
+		(fp_text user "*"
+			(at -4.7625 2.0828 0)
 			(layer "B.Fab")
 			(effects
@@
 			)
 		)
-		(fp_text user "*"
-			(at -4.7625 2.0828 0)
+		(fp_text user "ON"
+			(at 5.0165 5.1562 0)
 			(unlocked yes)
 			(layer "B.Fab")
@@
 			)
 		)
-		(fp_text user "OFF"
-			(at -5.0165 5.1562 0)
+		(fp_text user "*"
+			(at -4.7625 2.0828 0)
 			(unlocked yes)
 			(layer "B.Fab")
@@
 			)
 		)
-		(fp_text user "${REFERENCE}"
-			(at 0 4.7 0)
+		(fp_text user "OFF"
+			(at -5.0165 5.1562 0)
 			(unlocked yes)
 			(layer "B.Fab")
@@
 		(layer "B.Cu")
 		(at 127.15 68.6 180)
-		(property "Reference" "SW1"
+		(property "Reference" "PWR"
 			(at 7.55 0.1 90)
 			(layer "B.SilkS")
@@
 		(descr "LED SMD 0603 (1608 Metric), square (rectangular) end terminal, IPC-7351 nominal, (Body size source: http://www.tortai-tech.com/upload/download/2011102023233369053.pdf), generated with kicad-footprint-generator")
 		(tags "LED")
-		(property "Reference" "D2"
+		(property "Reference" "3v3"
 			(at 0 1.5 0)
 			(layer "B.SilkS")
@@
 		(layer "B.Cu")
 		(at 127.05 58.15)
-		(property "Reference" "SW3"
+		(property "Reference" "RESET"
 			(at -7.55 0.05 270)
 			(layer "B.SilkS")
@@
 		(descr "LED SMD 0603 (1608 Metric), square (rectangular) end terminal, IPC-7351 nominal, (Body size source: http://www.tortai-tech.com/upload/download/2011102023233369053.pdf), generated with kicad-footprint-generator")
 		(tags "LED")
-		(property "Reference" "D1"
-			(at 0.3 1.5 270)
+		(property "Reference" "PWR"
+			(at 0 1.5 90)
 			(layer "B.SilkS")
 			(effects
@@
 		)
 		(property "Value" "LED"
-			(at 0 -1.43 270)
+			(at 0 -1.43 90)
 			(layer "B.Fab")
 			(effects
@@
 		)
 		(property "Datasheet" "~"
-			(at 0 0 270)
+			(at 0 0 90)
 			(layer "B.Fab")
 			(hide yes)
@@
 		)
 		(property "Description" "Light emitting diode"
-			(at 0 0 270)
+			(at 0 0 90)
 			(layer "B.Fab")
 			(hide yes)
@@
 		)
 		(fp_text user "${REFERENCE}"
-			(at 0 0 270)
+			(at 0 0 90)
 			(layer "B.Fab")
 			(effects
@@
 		(layer "B.Cu")
 		(at 127.15 64 180)
-		(property "Reference" "SW2"
+		(property "Reference" "BOOT"
 			(at 7.65 0 90)
 			(layer "B.SilkS")

Commit message: v0.3.6
Parts:
- removed PWR: LED, LED_SMD:LED_0603_1608Metric
- added D1: PWR, LED_SMD:LED_0603_1608Metric, B.Cu at (163.3, 113.3)
- added D7: D_TVS, Diode_SMD:D_SOD-523, B.Cu at (161.8, 107.3)
- added F1: Polyfuse, Fuse:Fuse_1206_3216Metric, B.Cu at (162.5, 109.7)
- C20: moved to B.Cu
- D2: renamed from 3v3; value LED -> 3v3
- R5, R6, R8: value 65 -> 150
- R7: value 150 -> 348
- moved R7 44.9 mm to (163.3, 115.1), turned to 0 degrees
- moved C11 34.9 mm to (137.2, 101.1)
- moved C3 34.9 mm to (149.4, 99.5)
- moved IC1 34.9 mm to (151.3, 86.8)
- moved J2 34.9 mm to (154.4, 115.5)
- moved C10 34.9 mm to (137.2, 92.5)
- moved C18 34.9 mm to (152.3, 86.7)
- moved C5 34.9 mm to (140.7, 92.5)
- moved C6 34.9 mm to (141.6, 101.1)
- moved D3 34.9 mm to (146.7, 97.9)
- moved J1 34.9 mm to (140.6, 115.5)
- moved J5 34.9 mm to (168.1, 83.0)
- moved R10 34.9 mm to (147.4, 84.6)
- moved R11 34.9 mm to (145.4, 84.6)
- moved R17 34.9 mm to (125.5, 102.8)
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- renumbered PWR to SW1, BOOT to SW2, RESET to SW3
Connections:
- J6 pad 2: VDD -> Net-(J6-Pin_2)
Routing:
- net VDD: track 126.5 -> 112.8 mm
- net Net-(J6-Pin_2): track 0.00 -> 4.92 mm
- net Net-(D1-K): track 1.89 -> 2.47 mm
- net GND: track 48.6 -> 48.7 mm, vias 24 -> 25

Commit message: v0.3.7
Routing:
- net VDDA: track 48.7 -> 49.6 mm
Changed lines of the file:
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@@
 		)
 		(property "Value" "3v3"
-			(at 0 -1.43 0)
-			(layer "B.Fab")
+			(at 0 1.5 0)
+			(unlocked yes)
+			(layer "B.SilkS")
 			(effects
 				(font
@@
 			)
 		)
-		(property "Value" "3v3"
-			(at 0 1.5 0)
-			(unlocked yes)
-			(layer "B.SilkS")
-			(effects
-				(font
-					(size 1 1)
-					(thickness 0.15)
-				)
-				(justify mirror)
-			)
-		)
 		(property ki_fp_filters "LED* LED_SMD:* LED_THT:*")
 		(sheetname "/")
@@
 	)
 	(segment
+		(start 130.3 105.2)
+		(end 125 105.2)
+		(width 0.5)
+		(layer "In2.Cu")
+		(net 9)
+	)
+	(segment
 		(start 130.3 92.575)
 		(end 130.3 96.475)
@@
 	)
 	(segment
-		(start 132.475 102.075)
-		(end 137.967101 102.075)
+		(start 130.3 105.2)
+		(end 132.325 107.225)
 		(width 0.5)
 		(layer "In2.Cu")
@@
 	)
 	(segment
-		(start 130.3 99.9)
-		(end 124.425 105.775)
+		(start 132.325 107.225)
+		(end 134.3 107.225)
 		(width 0.5)
 		(layer "In2.Cu")
@@
 	)
 	(segment
-		(start 132.475 102.075)
-		(end 132.475 105.4)
+		(start 136.4 102.4)
+		(end 136.4 105.2)
 		(width 0.5)
 		(layer "In2.Cu")
@@
 	)
 	(segment
+		(start 136.725 102.075)
+		(end 136.4 102.4)
+		(width 0.5)
+		(layer "In2.Cu")
+		(net 9)
+	)
+	(segment
+		(start 134.375 107.225)
+		(end 134.3 107.225)
+		(width 0.3)
+		(layer "In2.Cu")
+		(net 9)
+	)
+	(segment
 		(start 137.117101 92.575)
 		(end 138.017101 93.475)
@@
 	)
 	(segment
+		(start 130.3 99.9)
+		(end 130.3 105.2)
+		(width 0.5)
+		(layer "In2.Cu")
+		(net 9)
+	)
+	(segment
 		(start 130.3 92.575)
 		(end 137.117101 92.575)
@@
 	)
 	(segment
-		(start 132.475 105.4)
-		(end 134.3 107.225)
+		(start 125 105.2)
+		(end 124.425 105.775)
 		(width 0.5)
 		(layer "In2.Cu")
@@
 	)
 	(segment
-		(start 130.3 99.9)
-		(end 132.475 102.075)
+		(start 137.967101 102.075)
+		(end 136.725 102.075)
+		(width 0.5)
+		(layer "In2.Cu")
+		(net 9)
+	)
+	(segment
+		(start 136.4 105.2)
+		(end 134.375 107.225)
 		(width 0.5)
 		(layer "In2.Cu")

Commit message: v0.3.8
Other:
- board text added: "3v3"
- board text added: "CLK"
- board text added: "GND"
- board text added: "IO"
- board text added: "RX"
- board text added: "TX"
- board text added: "VDD"
Changed lines of the file:
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@@
 		(tags "TSOT TO_SOT_SMD")
 		(property "Reference" "U7"
-			(at 0 -2.6 0)
+			(at 1.6 -2.525 0)
 			(layer "F.SilkS")
 			(effects
@@
 			(at 3.75 3.55 0)
 			(layer "B.SilkS")
+			(hide yes)
 			(effects
 				(font
@@
 			(layer "B.Fab")
 		)
-		(fp_text user "ON"
-			(at 5.0165 5.1562 0)
-			(unlocked yes)
-			(layer "B.SilkS")
-			(effects
-				(font
-					(size 1 1)
-					(thickness 0.15)
-				)
-				(justify mirror)
-			)
-		)
-		(fp_text user "OFF"
-			(at -5.0165 5.1562 0)
-			(unlocked yes)
-			(layer "B.SilkS")
-			(effects
-				(font
-					(size 1 1)
-					(thickness 0.15)
-				)
-				(justify mirror)
-			)
-		)
-		(fp_text user "CAN TERM"
+		(fp_text user "CAN-TERM"
 			(at 0 4.7 0)
 			(unlocked yes)
@@
 			(at 9.4 3.675 0)
 			(layer "B.SilkS")
+			(hide yes)
 			(effects
 				(font
@@
 			(at 7.55 0.1 90)
 			(layer "B.SilkS")
+			(hide yes)
 			(effects
 				(font
@@
 			)
 		)
+		(property "Field4" "PWR"
+			(at 7.65 -0.000001 90)
+			(unlocked yes)
+			(layer "B.SilkS")
+			(effects
+				(font
+					(size 1 1)
+					(thickness 0.15)
+				)
+				(justify mirror)
+			)
+		)
 		(sheetname "/")
 		(sheetfile "encoder.kicad_sch")
@@
 			(at -7.55 0.05 270)
 			(layer "B.SilkS")
+			(hide yes)
 			(effects
 				(font
@@
 			)
 		)
+		(property "Field4" "RESET"
+			(at -7.55 0 90)
+			(unlocked yes)
+			(layer "B.SilkS")
+			(effects
+				(font
+					(size 1 1)
+					(thickness 0.15)
+				)
+				(justify mirror)
+			)
+		)
 		(sheetname "/")
 		(sheetfile "encoder.kicad_sch")
@@
 			(at 7.65 0 90)
 			(layer "B.SilkS")
+			(hide yes)
 			(effects
 				(font
@@
 			)
 		)
+		(property "Value" "BOOT"
+			(at 7.65 -0.000001 90)
+			(unlocked yes)
+			(layer "B.SilkS")
+			(effects
+				(font
+					(size 1 1)
+					(thickness 0.15)
+				)
+				(justify mirror)
+			)
+		)
 		(sheetname "/")
 		(sheetfile "encoder.kicad_sch")
@@
 		(tags "connector JST XH vertical")
 		(property "Reference" "J3"
-			(at 3.75 3.55 0)
+			(at 7.6 3.6 0)
 			(layer "B.SilkS")
 			(effects
@@
 		)
 	)
+	(gr_text "GND"
+		(at 134.3 112.4 0)
+		(layer "B.SilkS")
+		(effects
+			(font
+				(size 1 1)
+				(thickness 0.15)
+			)
+			(justify left bottom mirror)
+		)
+	)
+	(gr_text "GND"
+		(at 147.9 112.5 0)
+		(layer "B.SilkS")
+		(effects
+			(font
+				(size 1 1)
+				(thickness 0.15)
+			)
+			(justify left bottom mirror)
+		)
+	)
+	(gr_text "IO\n"
+		(at 136.335317 112.4 0)
+		(layer "B.SilkS")
+		(effects
+			(font
+				(size 1 1)
+				(thickness 0.15)
+			)
+			(justify left bottom mirror)
+		)
+	)
+	(gr_text "VDD"
+		(at 156.625 112.5 0)
+		(layer "B.SilkS")
+		(effects
+			(font
+				(size 1 1)
+				(thickness 0.15)
+			)
+			(justify left bottom mirror)
+		)
+	)
+	(gr_text "CLK"
+		(at 139.656349 112.4 0)
+		(layer "B.SilkS")
+		(effects
+			(font
+				(size 1 1)
+				(thickness 0.15)
+			)
+			(justify left bottom mirror)
+		)
+	)
+	(gr_text "VDD"
+		(at 143.025 112.4 0)
+		(layer "B.SilkS")
+		(effects
+			(font
+				(size 1 1)
+				(thickness 0.15)
+			)
+			(justify left bottom mirror)
+		)
+	)
 	(gr_text "WANDA r1.0\n"
 		(at 139.7 109.757357 0)
@@
 			)
 			(justify left bottom mirror)
+		)
+	)
+	(gr_text "RX"
+		(at 150.586111 112.5 0)
+		(layer "B.SilkS")
+		(effects
+			(font
+				(size 1 1)
+				(thickness 0.15)
+			)
+			(justify left bottom mirror)
+		)
+	)
+	(gr_text "TX"
+		(at 153.034127 112.5 0)
+		(layer "B.SilkS")
+		(effects
+			(font
+				(size 1 1)
+				(thickness 0.15)
+			)
+			(justify left bottom mirror)
+		)
+	)
+	(gr_text "3v3"
+		(at 135.158334 88.7 0)
+		(layer "B.SilkS")
+		(effects
+			(font
+				(size 1 1)
+				(thickness 0.15)
+			)
+			(justify left bottom mirror)

Commit message: Fixed the PCB color
Parts:
- SW2: value SW_SPST -> BOOT
Changed lines of the file:
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@@
 			(layer "F.SilkS"
 				(type "Top Silk Screen")
-				(color "White")
+				(color "Black")
 			)
 			(layer "F.Paste"
@@
 			(layer "F.Mask"
 				(type "Top Solder Mask")
-				(color "Black")
+				(color "White")
 				(thickness 0.01)
 			)
@@
 			(layer "dielectric 1"
 				(type "prepreg")
+				(color "FR4 natural")
 				(thickness 0.1)
 				(material "FR4")
@@
 			(layer "dielectric 2"
 				(type "core")
+				(color "FR4 natural")
 				(thickness 1.24)
 				(material "FR4")
@@
 			(layer "dielectric 3"
 				(type "prepreg")
+				(color "FR4 natural")
 				(thickness 0.1)
 				(material "FR4")
@@
 			(layer "B.Mask"
 				(type "Bottom Solder Mask")
-				(color "Black")
+				(color "White")
 				(thickness 0.01)
 			)
@@
 			(layer "B.SilkS"
 				(type "Bottom Silk Screen")
-				(color "White")
+				(color "Black")
 			)
 			(copper_finish "None")
@@
 			)
 		)
-		(property "Value" "SW_SPST"
-			(at 10.97 -2.885 0)
-			(layer "B.Fab")
+		(property "Value" "BOOT"
+			(at 7.65 -0.000001 90)
+			(unlocked yes)
+			(layer "B.SilkS")
 			(effects
 				(font
@@
 					(thickness 0.15)
 				)
-				(justify mirror)
-			)
-		)
-		(property "Value" "BOOT"
-			(at 7.65 -0.000001 90)
-			(unlocked yes)
-			(layer "B.SilkS")
-			(effects
-				(font
-					(size 1 1)
-					(thickness 0.15)
-				)
