File: boards/encoder/psu.kicad_sch (KiCad schematic)
At the start: 10 parts, among them J1 Conn_PWR, U2 TPS62A02A

Commit message: v0.1.18
Parts:
- J6: renamed from J1; value Conn_PWR -> PWR
- renumbered C1 to C19, C2 to C20, C3 to C21, C4 to C22, R1 to R31, R2 to R32, U2 to U9
Other:
- note added: "Feedback loop"
- note added: "SMPS Components"
- company: (none) -> MetisVela
- title: (none) -> Wanda
- moved on the sheet: C19, C20, C21, C22, J6, L1, R31, R32, RV1, U9

Commit message: Fixed some values
Parts:
- R32: value 90k -> 95k
Changed lines of the file:
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@@
 			)
 		)
-		(property "Value" "90k"
+		(property "Value" "95k"
 			(at 45.72 57.1499 0)
 			(effects

Commit message: v0.2.1
Parts:
- C19, C20, C21, C22: footprint (none) -> Capacitor_SMD:C_0603_1608Metric
- L1: footprint (none) -> Inductor_SMD:L_1210_3225Metric
- R31, R32: footprint (none) -> Resistor_SMD:R_0603_1608Metric
- U9: footprint SOT6_DRL_TEX -> Package_TO_SOT_SMD:SOT-563
Other:
- moved on the sheet: C19
Changed lines of the file:
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@@
+	(wire
+		(pts
+			(xy 43.18 40.64) (xy 43.18 41.91)
+		)
+		(stroke
+			(width 0)
+			(type default)
+		)
+	)
 	(wire
 		(pts
@@
 	(wire
 		(pts
+			(xy 110.49 101.6) (xy 114.3 101.6)
+		)
+		(stroke
+			(width 0)
+			(type default)
+		)
+	)
+	(wire
+		(pts
+			(xy 90.17 99.06) (xy 95.25 99.06)
+		)
+		(stroke
+			(width 0)
+			(type default)
+		)
+	)
+	(wire
+		(pts
+			(xy 71.12 102.87) (xy 71.12 105.41)
+		)
+		(stroke
+			(width 0)
+			(type default)
+		)
+	)
+	(wire
+		(pts
 			(xy 43.18 41.91) (xy 43.18 43.18)
 		)
@@
 	(wire
 		(pts
-			(xy 110.49 101.6) (xy 114.3 101.6)
-		)
-		(stroke
-			(width 0)
-			(type default)
-		)
-	)
-	(wire
-		(pts
-			(xy 90.17 99.06) (xy 95.25 99.06)
-		)
-		(stroke
-			(width 0)
-			(type default)
-		)
-	)
-	(wire
-		(pts
-			(xy 71.12 102.87) (xy 71.12 105.41)
-		)
-		(stroke
-			(width 0)
-			(type default)
-		)
-	)
-	(wire
-		(pts
-			(xy 43.18 40.64) (xy 43.18 41.91)
+			(xy 53.34 41.91) (xy 53.34 40.64)
 		)
 		(stroke
@@
 	(wire
 		(pts
-			(xy 53.34 34.29) (xy 53.34 31.75)
+			(xy 53.34 33.02) (xy 53.34 31.75)
 		)
 		(stroke
@@
 			)
 		)
-		(property "Footprint" ""
+		(property "Footprint" "Resistor_SMD:R_0603_1608Metric"
 			(at 41.402 36.83 90)
 			(effects
@@
 	(symbol
 		(lib_id "Device:C")
-		(at 53.34 38.1 0)
+		(at 53.34 36.83 0)
 		(unit 1)
 		(exclude_from_sim no)
@@
 		(fields_autoplaced yes)
 		(property "Reference" "C19"
-			(at 57.15 36.8299 0)
+			(at 57.15 35.5599 0)
 			(effects
 				(font
@@
 		)
 		(property "Value" "120p"
-			(at 57.15 39.3699 0)
+			(at 57.15 38.0999 0)
 			(effects
 				(font
@@
 			)
 		)
-		(property "Footprint" ""
-			(at 54.3052 41.91 0)
+		(property "Footprint" "Capacitor_SMD:C_0603_1608Metric"
+			(at 54.3052 40.64 0)
 			(effects
 				(font
@@
 		)
 		(property "Datasheet" "~"
-			(at 53.34 38.1 0)
+			(at 53.34 36.83 0)
 			(effects
 				(font
@@
 		)
 		(property "Description" "Unpolarized capacitor"
-			(at 53.34 38.1 0)
+			(at 53.34 36.83 0)
 			(effects
 				(font
@@
 			)
 		)
-		(property "Footprint" ""
+		(property "Footprint" "Capacitor_SMD:C_0603_1608Metric"
 			(at 46.6852 102.87 0)
 			(effects
@@
 			)
 		)
-		(property "Footprint" ""
+		(property "Footprint" "Inductor_SMD:L_1210_3225Metric"
 			(at 36.83 31.75 0)
 			(effects
@@
 			)
 		)
-		(property "Footprint" ""
+		(property "Footprint" "Capacitor_SMD:C_0603_1608Metric"
 			(at 72.0852 102.87 0)
 			(effects
@@
 			)
 		)
-		(property "Footprint" "SOT6_DRL_TEX"
+		(property "Footprint" "Package_TO_SOT_SMD:SOT-563"
 			(at 102.87 99.06 0)
 			(effects
@@
 			)
 		)
-		(property "Footprint" ""
+		(property "Footprint" "Resistor_SMD:R_0603_1608Metric"
 			(at 41.402 55.88 90)
 			(effects
@@
 			)
 		)
-		(property "Footprint" ""
+		(property "Footprint" "Capacitor_SMD:C_0603_1608Metric"
 			(at 59.3852 102.87 0)
 			(effects

Commit message: v0.2.3
Parts:
- RV1: footprint (none) -> Potentiometer_SMD:Potentiometer_Bourns_TC33X_Vertical
Changed lines of the file:
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@@
 			)
 		)
-		(property "Footprint" ""
+		(property "Footprint" "Potentiometer_SMD:Potentiometer_Bourns_TC33X_Vertical"
 			(at 43.18 46.99 0)
 			(effects

Commit message: v0.2.9
Parts:
- J6: footprint (none) -> Connector_JST:JST_XH_B2B-XH-A_1x02_P2.50mm_Vertical
- renumbered R31 to R29, R32 to R30, U9 to U10
Changed lines of the file:
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@@
 		(dnp no)
 		(fields_autoplaced yes)
-		(property "Reference" "#PWR087"
+		(property "Reference" "#PWR090"
 			(at 26.67 111.76 0)
 			(effects
@@
 			(project "encoder"
 				(path "/710faa81-ee23-422b-ba7e-b655a364ab6f/4eebcdb7-98fa-4c4e-819b-5b04763be839"
-					(reference "#PWR087")
+					(reference "#PWR090")
 					(unit 1)
 				)
@@
 		(on_board yes)
 		(dnp no)
-		(property "Reference" "R31"
+		(property "Reference" "R29"
 			(at 45.72 35.5599 0)
 			(effects
@@
 			(project "encoder"
 				(path "/710faa81-ee23-422b-ba7e-b655a364ab6f/4eebcdb7-98fa-4c4e-819b-5b04763be839"
-					(reference "R31")
+					(reference "R29")
 					(unit 1)
 				)
@@
 			)
 		)
-		(property "Footprint" ""
+		(property "Footprint" "Connector_JST:JST_XH_B2B-XH-A_1x02_P2.50mm_Vertical"
 			(at 34.29 97.79 0)
 			(effects
@@
 		(dnp no)
 		(fields_autoplaced yes)
-		(property "Reference" "#PWR080"
+		(property "Reference" "#PWR083"
 			(at 53.34 34.29 0)
 			(effects
@@
 			(project "encoder"
 				(path "/710faa81-ee23-422b-ba7e-b655a364ab6f/4eebcdb7-98fa-4c4e-819b-5b04763be839"
-					(reference "#PWR080")
+					(reference "#PWR083")
 					(unit 1)
 				)
@@
 		(dnp no)
 		(fields_autoplaced yes)
-		(property "Reference" "#PWR081"
+		(property "Reference" "#PWR084"
 			(at 43.18 67.31 0)
 			(effects
@@
 			(project "encoder"
 				(path "/710faa81-ee23-422b-ba7e-b655a364ab6f/4eebcdb7-98fa-4c4e-819b-5b04763be839"
-					(reference "#PWR081")
+					(reference "#PWR084")
 					(unit 1)
 				)
@@
 		(dnp no)
 		(fields_autoplaced yes)
-		(property "Reference" "#PWR085"
+		(property "Reference" "#PWR088"
 			(at 71.12 96.52 0)
 			(effects
@@
 			(project "encoder"
 				(path "/710faa81-ee23-422b-ba7e-b655a364ab6f/4eebcdb7-98fa-4c4e-819b-5b04763be839"
-					(reference "#PWR085")
+					(reference "#PWR088")
 					(unit 1)
 				)
@@
 		(dnp no)
 		(fields_autoplaced yes)
-		(property "Reference" "#PWR089"
+		(property "Reference" "#PWR092"
 			(at 58.42 111.76 0)
 			(effects
@@
 			(project "encoder"
 				(path "/710faa81-ee23-422b-ba7e-b655a364ab6f/4eebcdb7-98fa-4c4e-819b-5b04763be839"
-					(reference "#PWR089")
+					(reference "#PWR092")
 					(unit 1)
 				)
@@
 		(dnp no)
 		(fields_autoplaced yes)
-		(property "Reference" "#PWR091"
+		(property "Reference" "#PWR094"
 			(at 92.71 111.76 0)
 			(effects
@@
 			(project "encoder"
 				(path "/710faa81-ee23-422b-ba7e-b655a364ab6f/4eebcdb7-98fa-4c4e-819b-5b04763be839"
-					(reference "#PWR091")
+					(reference "#PWR094")
 					(unit 1)
 				)
@@
 		(dnp no)
 		(fields_autoplaced yes)
-		(property "Reference" "#PWR086"
+		(property "Reference" "#PWR089"
 			(at 92.71 96.52 0)
 			(effects
@@
 			(project "encoder"
 				(path "/710faa81-ee23-422b-ba7e-b655a364ab6f/4eebcdb7-98fa-4c4e-819b-5b04763be839"
-					(reference "#PWR086")
+					(reference "#PWR089")
 					(unit 1)
 				)
@@
 		(dnp no)
 		(fields_autoplaced yes)
-		(property "Reference" "#PWR083"
+		(property "Reference" "#PWR086"
 			(at 45.72 96.52 0)
 			(effects
@@
 			(project "encoder"
 				(path "/710faa81-ee23-422b-ba7e-b655a364ab6f/4eebcdb7-98fa-4c4e-819b-5b04763be839"
-					(reference "#PWR083")
+					(reference "#PWR086")
 					(unit 1)
 				)
@@
 		(dnp no)
 		(fields_autoplaced yes)
-		(property "Reference" "#PWR084"
+		(property "Reference" "#PWR087"
 			(at 58.42 96.52 0)
 			(effects
@@
 			(project "encoder"
 				(path "/710faa81-ee23-422b-ba7e-b655a364ab6f/4eebcdb7-98fa-4c4e-819b-5b04763be839"
-					(reference "#PWR084")
+					(reference "#PWR087")
 					(unit 1)
 				)
@@
 		(dnp no)
 		(fields_autoplaced yes)
-		(property "Reference" "#PWR090"
+		(property "Reference" "#PWR093"
 			(at 71.12 111.76 0)
 			(effects
@@
 			(project "encoder"
 				(path "/710faa81-ee23-422b-ba7e-b655a364ab6f/4eebcdb7-98fa-4c4e-819b-5b04763be839"
-					(reference "#PWR090")
+					(reference "#PWR093")
 					(unit 1)
 				)
@@
 		(dnp no)
 		(fields_autoplaced yes)
-		(property "Reference" "U9"
+		(property "Reference" "U10"
 			(at 102.87 88.9 0)
 			(effects
@@
 			(project "encoder"
 				(path "/710faa81-ee23-422b-ba7e-b655a364ab6f/4eebcdb7-98fa-4c4e-819b-5b04763be839"
-					(reference "U9")
+					(reference "U10")
 					(unit 1)
 				)
@@
 		(dnp no)
 		(fields_autoplaced yes)
-		(property "Reference" "R32"
+		(property "Reference" "R30"
 			(at 45.72 54.6099 0)
 			(effects
@@
 			(project "encoder"
 				(path "/710faa81-ee23-422b-ba7e-b655a364ab6f/4eebcdb7-98fa-4c4e-819b-5b04763be839"
-					(reference "R32")
+					(reference "R30")
 					(unit 1)
 				)
@@
 		(dnp no)
 		(fields_autoplaced yes)
-		(property "Reference" "#PWR082"
+		(property "Reference" "#PWR085"
 			(at 26.67 96.52 0)
 			(effects
@@
 			(project "encoder"
 				(path "/710faa81-ee23-422b-ba7e-b655a364ab6f/4eebcdb7-98fa-4c4e-819b-5b04763be839"
-					(reference "#PWR082")
+					(reference "#PWR085")
 					(unit 1)
 				)
@@
 		(dnp no)
 		(fields_autoplaced yes)
-		(property "Reference" "#PWR088"
+		(property "Reference" "#PWR091"
 			(at 45.72 111.76 0)
 			(effects
@@
 			(project "encoder"
 				(path "/710faa81-ee23-422b-ba7e-b655a364ab6f/4eebcdb7-98fa-4c4e-819b-5b04763be839"
-					(reference "#PWR088")
-					(unit 1)
-				)
+					(reference "#PWR091")
+					(unit 1)
+				)

Commit message: v0.3.0
Parts:
- C20: footprint Capacitor_SMD:C_0603_1608Metric -> Capacitor_SMD:C_1206_3216Metric
Connections:
- net GND: now also J6.1 (Pin_1); no longer J6.2 (Pin_2)
- net VDD: now also J6.2 (Pin_2); no longer J6.1 (Pin_1)
Changed lines of the file:
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@@
 	(symbol
 		(lib_id "Connector_Generic:Conn_01x02")
-		(at 34.29 97.79 0)
+		(at 34.29 100.33 0)
+		(mirror x)
 		(unit 1)
 		(exclude_from_sim no)
@@
 		(on_board yes)
 		(dnp no)
-		(fields_autoplaced yes)
 		(property "Reference" "J6"
-			(at 36.83 97.7899 0)
+			(at 38.608 97.79 0)
 			(effects
 				(font
 					(size 1.27 1.27)
 				)
-				(justify left)
+				(justify right)
 			)
 		)
 		(property "Value" "PWR"
-			(at 36.83 100.3299 0)
+			(at 40.132 100.33 0)
 			(effects
 				(font
 					(size 1.27 1.27)
 				)
-				(justify left)
+				(justify right)
 			)
 		)
 		(property "Footprint" "Connector_JST:JST_XH_B2B-XH-A_1x02_P2.50mm_Vertical"
-			(at 34.29 97.79 0)
+			(at 34.29 100.33 0)
 			(effects
 				(font
@@
 		)
 		(property "Datasheet" "~"
-			(at 34.29 97.79 0)
+			(at 34.29 100.33 0)
 			(effects
 				(font
@@
 		)
 		(property "Description" "Generic connector, single row, 01x02, script generated (kicad-library-utils/schlib/autogen/connector/)"
-			(at 34.29 97.79 0)
+			(at 34.29 100.33 0)
 			(effects
 				(font
@@
 			)
 		)
-		(property "Footprint" "Capacitor_SMD:C_0603_1608Metric"
+		(property "Footprint" "Capacitor_SMD:C_1206_3216Metric"
 			(at 46.6852 102.87 0)
 			(effects

Commit message: v0.3.6
Parts:
- added D7: D_TVS, Diode_SMD:D_SOD-523, symbol Device:D_TVS
- added F1: Polyfuse, Fuse:Fuse_1206_3216Metric, symbol Device:Polyfuse
Connections:
- net GND: now also D7.1 (A1)
- net VDD: now also D7.2 (A2), F1.1; no longer J6.2 (Pin_2)
- new net: F1.2, J6.2 (Pin_2)
Other:
- note added: "Surge protection"
- moved on the sheet: C20, C21, C22, J6, U10

Commit message: v0.3.10
Parts:
- C22: footprint Capacitor_SMD:C_0603_1608Metric -> Capacitor_SMD:C_1206_3216Metric
- R27: renamed from R29; value 455k -> 453k
- R28: renamed from R30; value 95k -> 95.3k
Changed lines of the file:
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@@
 		(on_board yes)
 		(dnp no)
-		(property "Reference" "R29"
+		(property "Reference" "R27"
 			(at 45.72 35.5599 0)
 			(effects
@@
 			)
 		)
-		(property "Value" "455k"
+		(property "Value" "453k"
 			(at 45.466 38.354 0)
 			(effects
@@
 			)
 		)
+		(property "Sim.Type" ""
+			(at 43.18 36.83 0)
+			(effects
+				(font
+					(size 1.27 1.27)
+				)
+				(hide yes)
+			)
+		)
 		(pin "1"
 		)
@@
 			(project "encoder"
 				(path "/710faa81-ee23-422b-ba7e-b655a364ab6f/4eebcdb7-98fa-4c4e-819b-5b04763be839"
-					(reference "R29")
+					(reference "R27")
 					(unit 1)
 				)
@@
 		)
 		(property "Description" "Unpolarized capacitor"
+			(at 53.34 36.83 0)
+			(effects
+				(font
+					(size 1.27 1.27)
+				)
+				(hide yes)
+			)
+		)
+		(property "Sim.Type" ""
 			(at 53.34 36.83 0)
 			(effects
@@
 			)
 		)
+		(property "Sim.Type" ""
+			(at 46.99 147.32 0)
+			(effects
+				(font
+					(size 1.27 1.27)
+				)
+				(hide yes)
+			)
+		)
 		(pin "2"
 		)
@@
 			)
 		)
+		(property "Sim.Type" ""
+			(at 26.67 99.06 0)
+			(effects
+				(font
+					(size 1.27 1.27)
+				)
+				(hide yes)
+			)
+		)
 		(pin "1"
 		)
@@
 			)
 		)
+		(property "Sim.Type" ""
+			(at 36.83 31.75 90)
+			(effects
+				(font
+					(size 1.27 1.27)
+				)
+				(hide yes)
+			)
+		)
 		(pin "1"
 		)
@@
 		(property "Description" "Bidirectional transient-voltage-suppression diode"
 			(at 26.67 146.05 0)
+			(effects
+				(font
+					(size 1.27 1.27)
+				)
+				(hide yes)
+			)
+		)
+		(property "Sim.Type" ""
+			(at 26.67 146.05 90)
 			(effects
 				(font
@@
 			)
 		)
+		(property "Sim.Type" ""
+			(at 43.18 46.99 0)
+			(effects
+				(font
+					(size 1.27 1.27)
+				)
+				(hide yes)
+			)
+		)
 		(pin "2"
 		)
@@
 			)
 		)
+		(property "Sim.Type" ""
+			(at 33.02 139.7 90)
+			(effects
+				(font
+					(size 1.27 1.27)
+				)
+				(hide yes)
+			)
+		)
 		(pin "1"
 		)
@@
 			)
 		)
-		(property "Footprint" "Capacitor_SMD:C_0603_1608Metric"
+		(property "Footprint" "Capacitor_SMD:C_1206_3216Metric"
 			(at 53.0352 102.87 0)
 			(effects
@@
 			)
 		)
+		(property "Sim.Type" ""
+			(at 52.07 99.06 0)
+			(effects
+				(font
+					(size 1.27 1.27)
+				)
+				(hide yes)
+			)
+		)
 		(pin "1"
 		)
@@
 			)
 		)
+		(property "Sim.Type" ""
+			(at 83.82 99.06 0)
+			(effects
+				(font
+					(size 1.27 1.27)
+				)
+				(hide yes)
+			)
+		)
 		(pin "6"
 		)
@@
 		(dnp no)
 		(fields_autoplaced yes)
-		(property "Reference" "R30"
+		(property "Reference" "R28"
 			(at 45.72 54.6099 0)
 			(effects
@@
 			)
 		)
-		(property "Value" "95k"
+		(property "Value" "95.3k"
 			(at 45.72 57.1499 0)
 			(effects
@@
 			)
 		)
+		(property "Sim.Type" ""
+			(at 43.18 55.88 0)
+			(effects
+				(font
+					(size 1.27 1.27)
+				)
+				(hide yes)
+			)
+		)
 		(pin "1"
 		)
@@
 			(project "encoder"
 				(path "/710faa81-ee23-422b-ba7e-b655a364ab6f/4eebcdb7-98fa-4c4e-819b-5b04763be839"
-					(reference "R30")
+					(reference "R28")
 					(unit 1)
 				)
@@
 			(at 39.37 99.06 0)
 			(effects
+				(font
+					(size 1.27 1.27)
+				)
+				(hide yes)
+			)
+		)
+		(property "Sim.Type" ""
+			(at 39.37 99.06 0)
+			(effects
