File: boards/encoder/psu.kicad_sch (KiCad schematic)
At the start: 12 parts, among them J6 PWR, U10 TPS62A02A

Commit message: v1.0.2
Parts:
- U10: footprint Package_TO_SOT_SMD:SOT-563 -> metis-vela:SOT6_DRL_TEX
Changed lines of the file:
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@@
 			)
 		)
-		(property "Footprint" "Package_TO_SOT_SMD:SOT-563"
+		(property "Footprint" "metis-vela:SOT6_DRL_TEX"
 			(at 83.82 99.06 0)
 			(hide yes)
